Commit message: Improved track definition

File: panther_description/urdf/gear.urdf.xacro (robot description, xacro)
@@ -19,14 +19,5 @@
   </link>
   <joint name="gear_${position}_joint" type="continuous">
-    <xacro:if value="${position == 'left'}">
-    <origin
-      xyz="0.0536535102814494 -0.00979339452125411 0.0186240655062149"
-      rpy="-1.5707963267949 -1.50760970347625 3.14159265358979" />
-    </xacro:if>
-    <xacro:if value="${position == 'right'}">
-    <origin
-      xyz="0.0536535102814494 0.00979339452125411 0.0186240655062149"
-      rpy="1.5707963267949 -1.50760970347625 3.14159265358979" />
-    </xacro:if>
+    <xacro:insert_block name="joint_pose"/>
     <parent link="track_${position}_link" />
     <child link="gear_${position}_Link" />

File: panther_description/urdf/panther.urdf.xacro (robot description, xacro)
@@ -53,26 +53,26 @@
   <!-- passive_wheel_type type: (1) continuous or (2) fixed -->
   <xacro:track name="Left" position="left" parent="frame_link" passive_wheel_type="fixed">
-    <origin xyz="0 -0.161 -0.014" rpy="0 0 0" />
+    <origin
+      xyz="0 -0.161 -0.014"
+      rpy="0 0 0" />
+    <origin
+      xyz="0.15476 -${0.020382 + 0.161} -${0.026643 + 0.014}"
+      rpy="${M_PI/2} -${M_PI/2} 0" />
+    <origin
+      xyz="0.0536535102814494 -0.00979339452125411 0.0186240655062149"
+      rpy="-${M_PI/2} -${M_PI/2} ${M_PI}" />
   </xacro:track>
   <xacro:track name="Right" position="right" parent="frame_link" passive_wheel_type="fixed">
-    <origin xyz="0 0.161 -0.014" rpy="0 0 0" />
+    <origin
+      xyz="0 0.161 -0.014"
+      rpy="0 0 0" />
+    <origin
+      xyz="0.15476 ${0.020382 + 0.161} -${0.026643 + 0.014}"
+      rpy="-${M_PI/2} -${M_PI/2} 0" />
+    <origin
+      xyz="0.0536535102814494 0.00979339452125411 0.0186240655062149"
+      rpy="${M_PI/2} -${M_PI/2} ${M_PI}" />
   </xacro:track>
   <!-- Track - END -->
-  <!-- Sprocket -->
-  <!--<xacro:sprocket name="Left" position="left" parent="track_left_link">
-    <origin xyz="0 -0.161 -0.014" rpy="0 0 0" />
-  </xacro:sprocket>
-  <xacro:sprocket name="Right" position="right" parent="track_right_link">
-    <origin xyz="0 0.161 -0.014" rpy="0 0 0" />
-  </xacro:sprocket>-->
-  <!-- Sprocket - END -->
-  <!-- Gear -->
-  <!--<xacro:gear name="Left" position="left" parent="track_left_link">
-    <origin xyz="0 -0.161 -0.014" rpy="0 0 0" />
-  </xacro:gear>
-  <xacro:gear name="Right" position="right" parent="track_right_link">
-    <origin xyz="0 0.161 -0.014" rpy="0 0 0" />
-  </xacro:gear>-->
-  <!-- Gear - END -->
   </xacro:macro>
 </robot>

File: panther_description/urdf/sprocket.urdf.xacro (robot description, xacro)
@@ -25,15 +25,6 @@
   </link>
   <joint name="${name}" type="continuous">
-    <xacro:if value="${position == 'left'}">
-    <origin
-      xyz="0.15476 -0.020382 -0.026643"
-      rpy="1.5708 -1.5708 0" />
-    </xacro:if>
-    <xacro:if value="${position == 'right'}">
-    <origin
-      xyz="0.15476 0.020382 -0.026643"
-      rpy="-1.5708 -1.5708 0" />
-    </xacro:if>
-    <parent link="track_${position}_link" />
+    <xacro:insert_block name="joint_pose"/>
+    <parent link="${parent}" />
     <child link="sprocket_${position}_Link" />
     <axis xyz="0 0 -1" />

File: panther_description/urdf/track.urdf.xacro (robot description, xacro)
@@ -2,5 +2,5 @@
 <robot xmlns:xacro="http://ros.org/wiki/xacro" name="track">
  <!-- passive_wheel_type tye: (1) continuous or (2) fixed -->
- <xacro:macro name="track" params="name position parent passive_wheel_type *joint_pose">
+ <xacro:macro name="track" params="name position parent passive_wheel_type *track_pose *joint_pose *gear_pose">
   <!-- TRACK FIXED LINKS -->
   <link name="track_${position}_link">
@@ -21,5 +21,5 @@
   </link>
   <joint name="track_${position}_joint" type="fixed">
-    <xacro:insert_block name="joint_pose"/>
+    <xacro:insert_block name="track_pose"/>
     <parent link="${parent}" />
     <child link="track_${position}_link" />
@@ -329,11 +329,11 @@
   </joint>
   <!-- Sprocket -->
-  <xacro:sprocket name="${name}" position="${position}" parent="track_${position}_link">
-    <origin xyz="0 -0.161 -0.014" rpy="0 0 0" />
+  <xacro:sprocket name="${name}" position="${position}" parent="${parent}">
+    <xacro:insert_block name="joint_pose"/>
   </xacro:sprocket>
   <!-- Sprocket - END -->
   <!-- Gear -->
   <xacro:gear name="${name}" position="${position}" parent="track_${position}_link">
-    <origin xyz="0 -0.161 -0.014" rpy="0 0 0" />
+    <xacro:insert_block name="gear_pose"/>
   </xacro:gear>
   <!-- Gear - END -->
