Commit message: clean and fix urdf

File: panther_description/urdf/gear.urdf.xacro (robot description, xacro)
@@ -1,8 +1,8 @@
 <?xml version="1.0"?>
 <robot xmlns:xacro="http://ros.org/wiki/xacro" name="gear">
- <xacro:macro name="gear" params="name position parent *joint_pose">
+ <xacro:macro name="gear" params="position parent *joint_pose">
   <link name="gear_${position}_Link">
     <inertial>
-      <origin xyz="0 0 0.008" rpy="0 0 0" />
+      <origin xyz="0 0 0.008" rpy="0 ${M_PI} 0" />
       <mass value="0.0111" />
       <inertia ixx="0" ixy="0" ixz="0"
@@ -11,5 +11,5 @@
     </inertial>
     <visual>
-      <origin xyz="0 0 0" rpy="0 0 0" />
+      <origin xyz="0 0 0" rpy="0 ${M_PI} 0" />
       <geometry>
         <mesh filename="${path_meshes}/track/gear_link.STL" />
@@ -24,5 +24,5 @@
     <axis xyz="0 0 -1" />
     <!-- Passive sprocket rotate automatically according to the status of the active one -->
-    <mimic joint="${name}" multiplier="${sprocket_teeth/gear_teeth}" offset="0"/>
+    <mimic joint="${position}_joint" multiplier="${sprocket_teeth/gear_teeth}" offset="0"/>
   </joint>
   </xacro:macro>

File: panther_description/urdf/panther.urdf.xacro (robot description, xacro)
@@ -72,40 +72,36 @@
   <!-- Chassis - END -->
   <!-- ZED -->
-  <xacro:zedcamera parent="frame_link">
+  <!--<xacro:zedcamera parent="frame_link">
     <origin xyz="0.03600 0 0.1900" rpy="0 0 -1.5707963267949" />
-  </xacro:zedcamera>
+  </xacro:zedcamera>-->
   <!-- ZED - END -->
   <!-- IMU -->
-  <xacro:imu name="base_imu" parent="frame_link">
+  <!--<xacro:imu name="base_imu" parent="frame_link">
     <origin xyz="0.0420817256507905 0 0.091441320597534" rpy="${M_PI} ${M_PI/2} 0" />
-    <!--<origin xyz="0.0420817256507905 0 0.091441320597534" rpy="${-M_PI/2} 0 ${M_PI/2}" />-->
-  </xacro:imu>
+  </xacro:imu>-->
   <!-- IMU -->
   <!-- Track -->
   <!-- passive_wheel_type type: (1) continuous or (2) fixed -->
-  <xacro:track name="left_joint" position="left" parent="frame_link" passive_wheel_type="fixed">
+  <xacro:track position="left" parent="frame_link" passive_wheel_type="continuous">
     <origin
       xyz="0 -0.161 -0.014"
       rpy="0 0 0" />
     <origin
-      xyz="0.15476 -${0.140618} -${0.026643 + 0.014}"
-      rpy="-${M_PI/2} ${M_PI/2} 0" />
-    <!--<origin
-      xyz="0.15476 -${0.020382 + 0.161} -${0.026643 + 0.014}"
-      rpy="-${M_PI/2} ${M_PI/2} 0" />-->
+      xyz="0.15476 -0.161 ${-0.014 - 0.0267}"
+      rpy="-${M_PI/2} 0 0" />
     <origin
-      xyz="0.0536535102814494 -0.00979339452125411 0.0186240655062149"
-      rpy="-${M_PI/2} -${M_PI/2} ${M_PI}" />
+      xyz="0.054 -0.010 0.019"
+      rpy="-${M_PI/2} 0 0" />
   </xacro:track>
-  <xacro:track name="right_joint" position="right" parent="frame_link" passive_wheel_type="fixed">
+  <xacro:track position="right" parent="frame_link" passive_wheel_type="continuous">
     <origin
       xyz="0 0.161 -0.014"
       rpy="0 0 0" />
     <origin
-      xyz="0.15476 ${0.020382 + 0.161} -${0.026643 + 0.014}"
-      rpy="-${M_PI/2} ${M_PI/2} 0" />
+      xyz="0.155 0.161 ${-0.014 - 0.0267}"
+      rpy="-${M_PI/2} 0 0" />
     <origin
-      xyz="0.0536535102814494 0.00979339452125411 0.0186240655062149"
-      rpy="${M_PI/2} -${M_PI/2} ${M_PI}" />
+      xyz="0.054 0.010 0.019"
+      rpy="${M_PI/2} 0 0" />
   </xacro:track>
   <!-- Track - END -->

File: panther_description/urdf/sprocket.urdf.xacro (robot description, xacro)
@@ -1,15 +1,40 @@
 <?xml version="1.0"?>
+<!--
+Copyright (C) 2017, Raffaello Bonghi <raffaello@rnext.it>
+All rights reserved
+Redistribution and use in source and binary forms, with or without
+modification, are permitted provided that the following conditions are met:
+1. Redistributions of source code must retain the above copyright
+   notice, this list of conditions and the following disclaimer.
+2. Redistributions in binary form must reproduce the above copyright
+   notice, this list of conditions and the following disclaimer in the
+   documentation and/or other materials provided with the distribution.
+3. Neither the name of the copyright holder nor the names of its
+   contributors may be used to endorse or promote products derived
+   from this software without specific prior written permission.
+THIS SOFTWARE IS PROVIDED BY THE COPYRIGHT HOLDERS AND
+CONTRIBUTORS "AS IS" AND ANY EXPRESS OR IMPLIED WARRANTIES, INCLUDING,
+BUT NOT LIMITED TO, THE IMPLIED WARRANTIES OF MERCHANTABILITY AND FITNESS
+FOR A PARTICULAR PURPOSE ARE DISCLAIMED. IN NO EVENT SHALL THE COPYRIGHT
+HOLDER OR CONTRIBUTORS BE LIABLE FOR ANY DIRECT, INDIRECT, INCIDENTAL,
+SPECIAL, EXEMPLARY, OR CONSEQUENTIAL DAMAGES (INCLUDING, BUT NOT LIMITED TO,
+PROCUREMENT OF SUBSTITUTE GOODS OR SERVICES; LOSS OF USE, DATA, OR PROFITS;
+OR BUSINESS INTERRUPTION) HOWEVER CAUSED AND ON ANY THEORY OF LIABILITY,
+WHETHER IN CONTRACT, STRICT LIABILITY, OR TORT (INCLUDING NEGLIGENCE
+OR OTHERWISE) ARISING IN ANY WAY OUT OF THE USE OF THIS SOFTWARE,
+EVEN IF ADVISED OF THE POSSIBILITY OF SUCH DAMAGE.
+-->
 <robot xmlns:xacro="http://ros.org/wiki/xacro" name="sprocket">
- <xacro:macro name="sprocket" params="name position parent *joint_pose">
+ <xacro:macro name="sprocket" params="position parent *joint_pose">
   <link name="sprocket_${position}_Link">
     <inertial>
-      <origin xyz="0 0 -0.0167" rpy="0 0 0" />
+      <origin xyz="0 0 ${-sprocket_leght / 2}" rpy="0 ${M_PI} 0" />
       <mass value="0.098" />
       <inertia ixx="0" ixy="0" ixz="0"
-        iyy="0" iyz="0"
-        izz="0" />
+                       iyy="0" iyz="0"
+                               izz="0" />
     </inertial>
     <visual>
-      <origin xyz="0 0 0" rpy="0 0 0" />
+      <origin xyz="0 0 ${-sprocket_leght / 2 + 0.005}" rpy="0 ${M_PI} 0" />
       <geometry>
         <mesh filename="${path_meshes}/track/sprocket_link.STL" />
@@ -18,5 +43,5 @@
     </visual>
     <collision>
-      <origin xyz="0 0 ${-sprocket_leght / 2}" rpy="0 0 0" />
+      <origin xyz="0 0 ${-sprocket_leght / 2}" rpy="0 ${M_PI} 0" />
       <geometry>
         <cylinder length="${sprocket_leght}" radius="${sprocket_radius}"/>
@@ -24,5 +49,5 @@
     </collision>
   </link>
-  <joint name="${name}" type="continuous">
+  <joint name="${position}_joint" type="continuous">
     <xacro:insert_block name="joint_pose"/>
     <parent link="${parent}" />
@@ -32,11 +57,10 @@
     <joint_properties damping="1.0" friction="1.0"/>
   </joint>
-  <transmission name="${name}_trans" type="SimpleTransmission">
+  <transmission name="${position}_trans" type="SimpleTransmission">
     <type>transmission_interface/SimpleTransmission</type>
-    <actuator name="${name}_motor">
+    <actuator name="${position}_motor">
       <mechanicalReduction>${gear_teeth/sprocket_teeth}</mechanicalReduction>
-      <!--<mechanicalReduction>1</mechanicalReduction>-->
     </actuator>
-    <joint name="${name}">
+    <joint name="${position}_joint">
       <hardwareInterface>hardware_interface/VelocityJointInterface</hardwareInterface>
     </joint>

File: panther_description/urdf/track.urdf.xacro (robot description, xacro)
@@ -27,5 +27,5 @@
 <robot xmlns:xacro="http://ros.org/wiki/xacro" name="track">
  <!-- passive_wheel_type tye: (1) continuous or (2) fixed -->
- <xacro:macro name="track" params="name position parent passive_wheel_type *track_pose *joint_pose *gear_pose">
+ <xacro:macro name="track" params="position parent passive_wheel_type *track_pose *joint_pose *gear_pose">
   <!-- TRACK FIXED LINKS -->
   <link name="track_${position}_link">
@@ -183,184 +183,220 @@
     <axis xyz="0 0 0" />
   </joint>
-  <!-- PASSIVE WHEELS -->
-  <link name="wheel_${position}_center_up_Link">
-    <inertial>
-      <origin xyz="0 0 0" rpy="0 0 0" />
-      <mass value="0.016" />
-      <inertia ixx="0" ixy="0" ixz="0"
-        iyy="0" iyz="0"
-        izz="0" />
-    </inertial>
-    <visual>
-      <origin xyz="0 0 0" rpy="0 0 0" />
-      <geometry>
-        <mesh filename="${path_meshes}/track/wheel_center_up_link.STL" />
-      </geometry>
-      <material name="White-Alpha" />
-    </visual>
-  </link>
-  <joint name="wheel_${position}_center_up_joint" type="${passive_wheel_type}">
-    <origin
-      xyz="0 0 0.0735790044064745"
-      rpy="1.5707963267949 -0.800774112020821 6.31428234397228E-17" />
-    <parent link="track_${position}_link" />
-    <child link="wheel_${position}_center_up_Link" />
-    <axis xyz="0 0 -1" />
-  </joint>
-  <link name="wheel_${position}_front_up_Link">
-    <inertial>
-      <origin xyz="0 0 -0.020143" rpy="0 0 0" />
-      <mass value="0.043" />
-      <inertia ixx="0" ixy="0" ixz="0"
-        iyy="0" iyz="0"
-        izz="0" />
-    </inertial>
-    <visual>
-      <origin xyz="0 0 0" rpy="0 0 0" />
-      <geometry>
-        <mesh filename="${path_meshes}/track/wheel_front_link.STL" />
-      </geometry>
-      <material name="White-Alpha" />
-    </visual>
-  </link>
-  <joint name="wheel_${position}_front_up_joint" type="${passive_wheel_type}">
-    <origin
-      xyz="-0.18867 -0.020143 0.010536"
-      rpy="-1.5708 -0.13483 3.1416" />
-    <parent link="track_${position}_link" />
-    <child link="wheel_${position}_front_up_Link" />
-    <axis xyz="0 0 -1" />
-  </joint>
-  <!-- Front passive wheel all time type continous -->
-  <link name="wheel_${position}_front_down_Link">
-    <inertial>
-      <origin xyz="0 0 -0.020143" rpy="0 0 0" />
-      <mass value="0.0431" />
-      <inertia ixx="0" ixy="0" ixz="0"
-        iyy="0" iyz="0"
-        izz="0" />
-    </inertial>
-    <visual>
-      <origin xyz="0 0 0" rpy="0 0 0" />
-      <geometry>
-        <mesh filename="${path_meshes}/track/wheel_front_link.STL" />
-      </geometry>
-      <material name="White-Alpha" />
-    </visual>
-    <collision>
-      <origin xyz="0 0 -0.025" rpy="0 0 0" />
-      <geometry>
-        <cylinder length="0.05" radius="0.025"/>
-      </geometry>
-    </collision>
-  </link>
-  <joint name="wheel_${position}_front_down_joint" type="continuous">
-    <origin
-      xyz="-0.15659 -0.020143 -0.034143"
-      rpy="1.5708 -0.36637 2.3494E-17" />
-    <parent link="track_${position}_link" />
-    <child link="wheel_${position}_front_down_Link" />
-    <axis xyz="0 0 -1" />
-  </joint>
-  <link name="wheel_${position}_center_A_Link">
-    <inertial>
-      <origin xyz="-0.064 -0.046 0.004" rpy="0 0 0" />
-      <mass value="0.0082" />
-      <inertia ixx="0" ixy="0" ixz="0"
-        iyy="0" iyz="0"
-        izz="0" />
-    </inertial>
-    <visual>
-      <origin xyz="0 0 0" rpy="0 0 0" />
-      <geometry>
-        <mesh filename="${path_meshes}/track/wheel_center_link.STL" />
-      </geometry>
-      <material name="White-Alpha" />
-    </visual>
-  </link>
-  <joint name="wheel_${position}_center_A_joint" type="${passive_wheel_type}">
-    <origin xyz="-0.065 -0.004 -0.042" rpy="1.5708 0 0" />
-    <parent link="track_${position}_link" />
-    <child link="wheel_${position}_center_A_Link" />.
-    <axis xyz="0 0 -1" />
-  </joint>
-  <link name="wheel_${position}_center_B_Link">
-    <inertial>
-      <origin xyz="-0.020 -0.0465 0.004" rpy="0 0 0" />
-      <mass value="0.0083" />
-      <inertia ixx="0" ixy="0" ixz="0"
-        iyy="0" iyz="0"
-        izz="0" />
-    </inertial>
-    <visual>
-      <origin xyz="0 0 0" rpy="0 0 0" />
-      <geometry>
-        <mesh filename="${path_meshes}/track/wheel_center_link.STL" />
-      </geometry>
-      <material name="White-Alpha" />
-    </visual>
-  </link>
-  <joint name="wheel_${position}_center_B_joint" type="${passive_wheel_type}">
-    <origin xyz="-0.020 -0.004 -0.042" rpy="1.5708 0 0" />
-    <parent link="track_${position}_link" />
-    <child link="wheel_${position}_center_B_Link" />
-    <axis xyz="0 0 -1" />
-  </joint>
-  <link name="wheel_${position}_center_C_Link">
-    <inertial>
-      <origin xyz="0.020 -0.0462 0.004" rpy="0 0 0" />
-      <mass value="0.0083" />
-      <inertia ixx="0" ixy="0" ixz="0"
-        iyy="0" iyz="0"
-        izz="0" />
-    </inertial>
-    <visual>
-      <origin
-        xyz="0 0 0"
-        rpy="0 0 0" />
-      <geometry>
-        <mesh filename="${path_meshes}/track/wheel_center_link.STL" />
-      </geometry>
-      <material name="White-Alpha" />
-    </visual>
-  </link>
-  <joint name="wheel_${position}_center_C_joint" type="${passive_wheel_type}">
-    <origin xyz="0.020 -0.004 -0.042" rpy="1.5708 0 0" />
-    <parent link="track_${position}_link" />
-    <child link="wheel_${position}_center_C_Link" />
-    <axis xyz="0 0 -1" />
-  </joint>
-  <link name="wheel_${position}_center_D_Link">
-    <inertial>
-      <origin xyz="0.0648 -0.0462 0.004" rpy="0 0 0" />
-      <mass value="0.0083" />
-      <inertia ixx="0" ixy="0" ixz="0"
-        iyy="0" iyz="0"
-        izz="0" />
-    </inertial>
-    <visual>
-      <origin xyz="0 0 0" rpy="0 0 0" />
-      <geometry>
-        <mesh filename="${path_meshes}/track/wheel_center_link.STL" />
-      </geometry>
-      <material name="White-Alpha" />
-    </visual>
-  </link>
-  <joint name="wheel_${position}_center_D_joint" type="${passive_wheel_type}">
-    <origin xyz="0.065 -0.004 -0.042" rpy="1.5707963267949 0 0" />
-    <parent link="track_${position}_link" />
-    <child link="wheel_${position}_center_D_Link" />
-    <axis xyz="0 0 -1" />
-  </joint>
   <!-- Sprocket -->
-  <xacro:sprocket name="${name}" position="${position}" parent="${parent}">
+  <xacro:sprocket position="${position}" parent="${parent}">
     <xacro:insert_block name="joint_pose"/>
   </xacro:sprocket>
   <!-- Sprocket - END -->
   <!-- Gear -->
-  <xacro:gear name="${name}" position="${position}" parent="track_${position}_link">
+  <xacro:gear position="${position}" parent="track_${position}_link">
     <xacro:insert_block name="gear_pose"/>
   </xacro:gear>
   <!-- Gear - END -->
+  <!-- PASSIVE WHEELS -->
+  <link name="wheel_${position}_center_up_Link">
+    <inertial>
+      <origin xyz="0 0 0" rpy="0 0 0" />
+      <mass value="0.016" />
+      <inertia ixx="0" ixy="0" ixz="0"
+                       iyy="0" iyz="0"
+                               izz="0" />
+    </inertial>
+    <visual>
+      <origin xyz="0 0 0" rpy="0 0 0" />
+      <geometry>
+        <mesh filename="${path_meshes}/track/wheel_center_up_link.STL" />
+      </geometry>
+      <material name="White-Alpha" />
+    </visual>
+  </link>
+  <joint name="wheel_${position}_center_up_joint" type="${passive_wheel_type}">
+    <origin
+      xyz="0 0 0.0735790044064745"
+      rpy="-${M_PI/2} 0 0" />
+    <parent link="track_${position}_link" />
+    <child link="wheel_${position}_center_up_Link" />
+    <axis xyz="0 0 -1" />
+    <xacro:if value="${passive_wheel_type == 'continuous'}">
+    <!-- Passive sprocket rotate automatically according to the status of the active one -->
+      <mimic joint="${position}_joint" multiplier="1" offset="0"/>
+    </xacro:if>
+  </joint>
+  <link name="wheel_${position}_front_up_Link">
+    <inertial>
+      <origin xyz="0 0 0.020143" rpy="0 0 0" />
+      <mass value="0.043" />
+      <inertia ixx="0" ixy="0" ixz="0"
+                       iyy="0" iyz="0"
+                               izz="0" />
+    </inertial>
+    <visual>
+      <origin xyz="0 0 0.020143" rpy="0 0 0" />
+      <geometry>
+        <mesh filename="${path_meshes}/track/wheel_front_link.STL" />
+      </geometry>
+      <material name="White-Alpha" />
+    </visual>
+  </link>
+  <joint name="wheel_${position}_front_up_joint" type="${passive_wheel_type}">
+    <origin
+      xyz="-0.18867 0 0.010536"
+      rpy="-${M_PI/2} 0 0" />
+    <parent link="track_${position}_link" />
+    <child link="wheel_${position}_front_up_Link" />
+    <axis xyz="0 0 -1" />
+    <xacro:if value="${passive_wheel_type == 'continuous'}">
+    <!-- Passive sprocket rotate automatically according to the status of the active one -->
+      <mimic joint="${position}_joint" multiplier="1" offset="0"/>
+    </xacro:if>
+  </joint>
+  <!-- Front passive wheel all time type continous -->
+  <link name="wheel_${position}_front_down_Link">
+    <inertial>
+      <origin xyz="0 0 0.020143" rpy="0 0 0" />
+      <mass value="0.0431" />
+      <inertia ixx="0" ixy="0" ixz="0"
+                       iyy="0" iyz="0"
+                               izz="0" />
+    </inertial>
+    <visual>
+      <origin xyz="0 0 0.020143" rpy="0 0 0" />
+      <geometry>
+        <mesh filename="${path_meshes}/track/wheel_front_link.STL" />
+      </geometry>
+      <material name="White-Alpha" />
+    </visual>
+    <collision>
+      <origin xyz="0 0 -0.025" rpy="0 0 0" />
+      <geometry>
+        <cylinder length="0.05" radius="0.025"/>
+      </geometry>
+    </collision>
+  </link>
+  <joint name="wheel_${position}_front_down_joint" type="${passive_wheel_type}">
+    <origin
+      xyz="-0.15659 0 -0.034143"
+      rpy="-${M_PI/2} 0 0" />
+    <parent link="track_${position}_link" />
+    <child link="wheel_${position}_front_down_Link" />
+    <axis xyz="0 0 -1" />
+    <xacro:if value="${passive_wheel_type == 'continuous'}">
+    <!-- Passive sprocket rotate automatically according to the status of the active one -->
+      <mimic joint="${position}_joint" multiplier="1" offset="0"/>
+    </xacro:if>
+  </joint>
+  <link name="wheel_${position}_center_A_Link">
+    <inertial>
+      <origin xyz="-0.064 -0.046 0.004" rpy="0 0 0" />
+      <mass value="0.0082" />
+      <inertia ixx="0" ixy="0" ixz="0"
+                       iyy="0" iyz="0"
+                               izz="0" />
+    </inertial>
+    <visual>
+      <origin xyz="0 0 0" rpy="0 0 0" />
+      <geometry>
+        <mesh filename="${path_meshes}/track/wheel_center_link.STL" />
+      </geometry>
+      <material name="White-Alpha" />
+    </visual>
+  </link>
+  <joint name="wheel_${position}_center_A_joint" type="${passive_wheel_type}">
+    <origin
+       xyz="-0.065 -0.004 -0.042"
+       rpy="-${M_PI/2} 0 0" />
+    <parent link="track_${position}_link" />
+    <child link="wheel_${position}_center_A_Link" />.
+    <axis xyz="0 0 -1" />
+    <xacro:if value="${passive_wheel_type == 'continuous'}">
+    <!-- Passive sprocket rotate automatically according to the status of the active one -->
+      <mimic joint="${position}_joint" multiplier="1" offset="0"/>
+    </xacro:if>
+  </joint>
+  <link name="wheel_${position}_center_B_Link">
+    <inertial>
+      <origin xyz="-0.020 -0.0465 0.004" rpy="0 0 0" />
+      <mass value="0.0083" />
+      <inertia ixx="0" ixy="0" ixz="0"
+                       iyy="0" iyz="0"
+                               izz="0" />
+    </inertial>
+    <visual>
+      <origin xyz="0 0 0" rpy="0 0 0" />
+      <geometry>
+        <mesh filename="${path_meshes}/track/wheel_center_link.STL" />
+      </geometry>
+      <material name="White-Alpha" />
+    </visual>
+  </link>
+  <joint name="wheel_${position}_center_B_joint" type="${passive_wheel_type}">
+    <origin
+       xyz="-0.020 -0.004 -0.042"
+       rpy="-${M_PI/2} 0 0" />
+    <parent link="track_${position}_link" />
+    <child link="wheel_${position}_center_B_Link" />
+    <axis xyz="0 0 -1" />
+    <xacro:if value="${passive_wheel_type == 'continuous'}">
+    <!-- Passive sprocket rotate automatically according to the status of the active one -->
+      <mimic joint="${position}_joint" multiplier="1" offset="0"/>
+    </xacro:if>
+  </joint>
+  <link name="wheel_${position}_center_C_Link">
+    <inertial>
+      <origin xyz="0.020 -0.0462 0.004" rpy="0 0 0" />
+      <mass value="0.0083" />
+      <inertia ixx="0" ixy="0" ixz="0"
+                       iyy="0" iyz="0"
+                               izz="0" />
+    </inertial>
+    <visual>
+      <origin
+        xyz="0 0 0"
+        rpy="0 0 0" />
+      <geometry>
+        <mesh filename="${path_meshes}/track/wheel_center_link.STL" />
+      </geometry>
+      <material name="White-Alpha" />
+    </visual>
+  </link>
+  <joint name="wheel_${position}_center_C_joint" type="${passive_wheel_type}">
+    <origin
+       xyz="0.020 -0.004 -0.042"
+       rpy="-${M_PI/2} 0 0" />
+    <parent link="track_${position}_link" />
+    <child link="wheel_${position}_center_C_Link" />
+    <axis xyz="0 0 -1" />
+    <xacro:if value="${passive_wheel_type == 'continuous'}">
+    <!-- Passive sprocket rotate automatically according to the status of the active one -->
+      <mimic joint="${position}_joint" multiplier="1" offset="0"/>
+    </xacro:if>
+  </joint>
+  <link name="wheel_${position}_center_D_Link">
+    <inertial>
+      <origin xyz="0.0648 -0.0462 0.004" rpy="0 0 0" />
+      <mass value="0.0083" />
+      <inertia ixx="0" ixy="0" ixz="0"
+                       iyy="0" iyz="0"
+                               izz="0" />
+    </inertial>
+    <visual>
+      <origin xyz="0 0 0" rpy="0 0 0" />
+      <geometry>
+        <mesh filename="${path_meshes}/track/wheel_center_link.STL" />
+      </geometry>
+      <material name="White-Alpha" />
+    </visual>
+  </link>
+  <joint name="wheel_${position}_center_D_joint" type="${passive_wheel_type}">
+    <origin
+       xyz="0.065 -0.004 -0.042"
+       rpy="-${M_PI/2} 0 0" />
+    <parent link="track_${position}_link" />
+    <child link="wheel_${position}_center_D_Link" />
+    <axis xyz="0 0 -1" />
+    <xacro:if value="${passive_wheel_type == 'continuous'}">
+    <!-- Passive sprocket rotate automatically according to the status of the active one -->
+      <mimic joint="${position}_joint" multiplier="1" offset="0"/>
+    </xacro:if>
+  </joint>
   </xacro:macro>
 </robot>
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