Commit message: fixed gear plot

File: panther_description/urdf/gear.urdf.xacro (robot description, xacro)
@@ -1,8 +1,33 @@
 <?xml version="1.0"?>
+<!--
+Copyright (C) 2017, Raffaello Bonghi <raffaello@rnext.it>
+All rights reserved
+Redistribution and use in source and binary forms, with or without
+modification, are permitted provided that the following conditions are met:
+1. Redistributions of source code must retain the above copyright
+   notice, this list of conditions and the following disclaimer.
+2. Redistributions in binary form must reproduce the above copyright
+   notice, this list of conditions and the following disclaimer in the
+   documentation and/or other materials provided with the distribution.
+3. Neither the name of the copyright holder nor the names of its
+   contributors may be used to endorse or promote products derived
+   from this software without specific prior written permission.
+THIS SOFTWARE IS PROVIDED BY THE COPYRIGHT HOLDERS AND
+CONTRIBUTORS "AS IS" AND ANY EXPRESS OR IMPLIED WARRANTIES, INCLUDING,
+BUT NOT LIMITED TO, THE IMPLIED WARRANTIES OF MERCHANTABILITY AND FITNESS
+FOR A PARTICULAR PURPOSE ARE DISCLAIMED. IN NO EVENT SHALL THE COPYRIGHT
+HOLDER OR CONTRIBUTORS BE LIABLE FOR ANY DIRECT, INDIRECT, INCIDENTAL,
+SPECIAL, EXEMPLARY, OR CONSEQUENTIAL DAMAGES (INCLUDING, BUT NOT LIMITED TO,
+PROCUREMENT OF SUBSTITUTE GOODS OR SERVICES; LOSS OF USE, DATA, OR PROFITS;
+OR BUSINESS INTERRUPTION) HOWEVER CAUSED AND ON ANY THEORY OF LIABILITY,
+WHETHER IN CONTRACT, STRICT LIABILITY, OR TORT (INCLUDING NEGLIGENCE
+OR OTHERWISE) ARISING IN ANY WAY OUT OF THE USE OF THIS SOFTWARE,
+EVEN IF ADVISED OF THE POSSIBILITY OF SUCH DAMAGE.
+-->
 <robot xmlns:xacro="http://ros.org/wiki/xacro" name="gear">
  <xacro:macro name="gear" params="type orientation">
   <link name="gear_${type}_Link">
     <inertial>
-      <origin xyz="0 0 0.008" rpy="0 ${M_PI} 0" />
+      <origin xyz="0 0 0.008" rpy="0 0 0" />
       <mass value="0.0111" />
       <inertia ixx="0" ixy="0" ixz="0"
@@ -11,5 +36,5 @@
     </inertial>
     <visual>
-      <origin xyz="0 0 0" rpy="0 ${M_PI} 0" />
+      <origin xyz="0 0 0" rpy="0 0 0" />
       <geometry>
         <mesh filename="${path_meshes}/track/gear_link.STL" />
@@ -20,6 +45,6 @@
   <joint name="gear_${type}_joint" type="continuous">
     <origin
-      xyz="-0.0536535102814494 -0.00979339452125411 0.0186240655062149"
-      rpy="-${M_PI/2} ${M_PI} ${M_PI}" />
+      xyz="-0.0536535102814494 ${orientation * -0.00979339452125411} 0.0186240655062149"
+      rpy="${orientation * M_PI/2} 0 0" />
     <parent link="track_${type}_link" />
     <child link="gear_${type}_Link" />

Commit message: Improved gabeo view

File: panther_description/urdf/gear.urdf.xacro (robot description, xacro)
@@ -59,4 +59,7 @@
     <mimic joint="${type}_joint" multiplier="${sprocket_teeth/gear_teeth}" offset="0"/>
   </joint>
+  <gazebo reference="gear_${type}_Link">
+    <material>Gazebo/DarkGrey</material>
+  </gazebo>
   </xacro:macro>
 </robot>

File: panther_description/urdf/sprocket.urdf.xacro (robot description, xacro)
@@ -64,4 +64,8 @@
   </joint>
   <!-- Transmission -->
+  <gazebo reference="sprocket_${type}_Link">
+    <material>Gazebo/Black</material>
+  </gazebo>
+  <!-- Transmission -->
   <transmission name="${type}_trans" type="SimpleTransmission">
     <type>transmission_interface/SimpleTransmission</type>

File: panther_description/urdf/track.urdf.xacro (robot description, xacro)
@@ -37,4 +37,25 @@
     <xacro:property name="orientation" value="1"/>
   </xacro:if>
+  <gazebo reference="track_${type}_Link">
+    <material>Gazebo/White</material>
+  </gazebo>
+  <gazebo reference="fender_${type}_Link">
+    <material>Gazebo/Black</material>
+  </gazebo>
+  <gazebo reference="chain_${type}_Link">
+    <material>Gazebo/DarkGrey</material>
+  </gazebo>
+  <gazebo reference="rubber_${type}_Link">
+    <material>Gazebo/Black</material>
+  </gazebo>
+  <gazebo reference="iron_${type}_Link">
+    <material>Gazebo/Grey</material>
+  </gazebo>
+  <gazebo reference="damper_${type}_Link">
+    <material>Gazebo/Black</material>
+  </gazebo>
+  <gazebo reference="damper_label_${type}_Link">
+    <material>Gazebo/Red</material>
+  </gazebo>
   <!-- TRACK FIXED LINKS -->
   <link name="track_${type}_link">

File: panther_description/urdf/wheel.urdf.xacro (robot description, xacro)
@@ -60,4 +60,7 @@
     </xacro:if>
   </joint>
+  <gazebo reference="wheel_${type}_${conf}_Link">
+    <material>Gazebo/WhiteGlow</material>
+  </gazebo>
   </xacro:macro>
 </robot>
