Commit message: Added zed frames joint

File: panther_description/urdf/zedcamera.urdf.xacro (robot description, xacro)
@@ -1,4 +1,6 @@
 <?xml version="1.0"?>
 <robot name="zedcamera" xmlns:xacro="http://ros.org/wiki/xacro">
+<xacro:property name="optical_y_offset" value="0.06" />
+<xacro:property name="optical_x_offset" value="0.03" />
   <xacro:macro name="zedcamera" params="parent *joint_pose">
   <link name="zed_stand_link">
@@ -24,5 +26,5 @@
     <axis xyz="0 0 0" />
   </joint>
-  <link name="zed_Link">
+  <link name="zed_camera_link">
     <inertial>
       <origin xyz="0 0 0.016" rpy="0 0 0" />
@@ -40,10 +42,34 @@
     </visual>
   </link>
-  <joint name="zed_joint" type="fixed">
+  <joint name="zed_camera_joint" type="fixed">
     <origin xyz="0 0 0" rpy="1.5707963267949 0 0" />
     <parent link="zed_stand_link" />
-    <child link="zed_Link" />
+    <child link="zed_camera_link" />
     <axis xyz="0 0 0" />
   </joint>
+    <joint name="zed_left_joint" type="fixed">
+      <origin xyz="${optical_y_offset} 0 ${optical_x_offset}" rpy="${-M_PI/2} ${-M_PI/2} 0"/>
+      <parent link="zed_camera_link"/>
+      <child link="zed_left_frame" />
+    </joint>
+    <link name="zed_left_frame"/>
+    <joint name="zed_left_optical_joint" type="fixed">
+      <origin xyz="0 0 0" rpy="${-M_PI/2} 0 ${-M_PI/2}" />
+      <parent link="zed_left_frame" />
+      <child link="zed_left_optical_frame" />
+    </joint>
+    <link name="zed_left_optical_frame"/>
+    <joint name="zed_right_joint" type="fixed">
+      <origin xyz="${-optical_y_offset} 0 ${optical_x_offset}" rpy="${-M_PI/2} ${-M_PI/2} 0"/>
+      <parent link="zed_camera_link" />
+      <child link="zed_right_frame" />
+    </joint>
+    <link name="zed_right_frame"/>
+    <joint name="zed_right_optical_joint" type="fixed">
+      <origin xyz="0 0 0" rpy="${-M_PI/2} 0 ${-M_PI/2}" />
+      <parent link="zed_right_frame" />
+      <child link="zed_right_optical_frame" />
+    </joint>
+    <link name="zed_right_optical_frame"/>
   </xacro:macro>
 </robot>

Commit message: Added IMU and diagnostic controller. minor fixes

File: panther_description/urdf/zedcamera.urdf.xacro (robot description, xacro)
@@ -73,4 +73,11 @@
     <parent link="zed_camera_link" />
     <child link="zed_initial_frame" />
+    <axis xyz="0 0 0" />
+  </joint>
+  <link name="zed_current_frame" />
+  <joint name="zed_current_joint" type="fixed">
+    <origin xyz="0 0.0 0" rpy="0 0 0" />
+    <parent link="zed_initial_frame" />
+    <child link="zed_current_frame" />
     <axis xyz="0 0 0" />
   </joint>

Commit message: Fixed some erroneus reference with ZED stl

File: panther_description/urdf/zedcamera.urdf.xacro (robot description, xacro)
@@ -55,5 +55,5 @@
       <origin xyz="0 0 0" rpy="0 0 0"/>
       <geometry>
-        <mesh filename="package://zed_wrapper/urdf/ZED.stl" />
+        <mesh filename="${path_meshes}/zed/ZED.stl" />
       </geometry>
       <material name="light_grey">
@@ -122,72 +122,4 @@
       <origin xyz="0 -0.12 0" rpy="0 0 0" />
   </joint>
-<!--  <link name="zed_stand_link">
-    <inertial>
-      <origin xyz="0 -0.0184 0.0173" rpy="0 0 0" />
-      <mass value="0.0173" />
-      <inertia ixx="2.76959607332778E-06" ixy="-7.16716953193216E-11" ixz="-1.34923517166624E-10"
-        iyy="6.44872593702919E-06" iyz="6.78675778442728E-08"
-        izz="4.02458373877404E-06" />
-    </inertial>
-    <visual>
-      <origin xyz="0 0 0" rpy="0 0 0" />
-      <geometry>
-        <mesh filename="${path_meshes}/zed/stand_link.STL" />
-      </geometry>
-      <material name="Black" />
-    </visual>
-  </link>
-  <joint name="zed_stand_sensor" type="fixed">
-    <xacro:insert_block name="joint_pose"/>
-    <parent link="${parent}" />
-    <child link="zed_stand_link" />
-    <axis xyz="0 0 0" />
-  </joint>
-  <link name="zed_camera_link">
-    <inertial>
-      <origin xyz="0 0 0.016" rpy="0 0 0" />
-      <mass value="0.6031" />
-      <inertia ixx="9.23924784521736E-05" ixy="2.60198941057937E-12" ixz="1.09417755562675E-13"
-        iyy="0.00146233786235907" iyz="3.89711252858911E-08"
-        izz="0.00144603978576908" />
-    </inertial>
-    <visual>
-      <origin xyz="0 0 0" rpy="0 0 0" />
-      <geometry>
-        <mesh filename="${path_meshes}/zed/zed_link.STL" />
-      </geometry>
-      <material name="Grey" />
-    </visual>
-  </link>
-  <joint name="zed_camera_joint" type="fixed">
-    <origin xyz="0 0 0" rpy="1.5707963267949 0 0" />
-    <parent link="zed_stand_link" />
-    <child link="zed_camera_link" />
-    <axis xyz="0 0 0" />
-  </joint>
-    <joint name="zed_left_joint" type="fixed">
-      <origin xyz="${optical_y_offset} 0 ${optical_x_offset}" rpy="${-M_PI/2} ${-M_PI/2} 0"/>
-      <parent link="zed_camera_link"/>
-      <child link="zed_left_frame" />
-    </joint>
-    <link name="zed_left_frame"/>
-    <joint name="zed_left_optical_joint" type="fixed">
-      <origin xyz="0 0 0" rpy="${-M_PI/2} 0 ${-M_PI/2}" />
-      <parent link="zed_left_frame" />
-      <child link="zed_left_optical_frame" />
-    </joint>
-    <link name="zed_left_optical_frame"/>
-    <joint name="zed_right_joint" type="fixed">
-      <origin xyz="${-optical_y_offset} 0 ${optical_x_offset}" rpy="${-M_PI/2} ${-M_PI/2} 0"/>
-      <parent link="zed_camera_link" />
-      <child link="zed_right_frame" />
-    </joint>
-    <link name="zed_right_frame"/>
-    <joint name="zed_right_optical_joint" type="fixed">
-      <origin xyz="0 0 0" rpy="${-M_PI/2} 0 ${-M_PI/2}" />
-      <parent link="zed_right_frame" />
-      <child link="zed_right_optical_frame" />
-    </joint>
-    <link name="zed_right_optical_frame"/>-->
   </xacro:macro>
 </robot>
