Commit message: minor fixes IMU

File: panther_description/urdf/imu.urdf.xacro (robot description, xacro)
@@ -27,5 +27,5 @@
 <robot xmlns:xacro="http://ros.org/wiki/xacro" name="imu">
   <xacro:macro name="imu" params="name parent *joint_pose">
-    <link name="${name}_link">
+    <link name="${name}_center_link">
       <inertial>
         <origin xyz="0.0002 0.003 -0.00025" rpy="0 0 0" />
@@ -33,6 +33,6 @@
         <inertia
           ixx="6.80127923442653E-07" ixy="2.58853590724977E-08" ixz="6.27330058259111E-09"
-          iyy="2.67621227004883E-07" iyz="3.00971478682596E-08"
-          izz="9.29933868272119E-07" />
+                                     iyy="2.67621227004883E-07" iyz="3.00971478682596E-08"
+                                                                izz="9.29933868272119E-07" />
       </inertial>
       <visual>
@@ -44,7 +44,13 @@
       </visual>
     </link>
-    <joint name="${name}_joint" type="fixed">
+    <joint name="${name}_center_joint" type="fixed">
       <xacro:insert_block name="joint_pose"/>
       <parent link="${parent}" />
+      <child link="${name}_center_link" />
+    </joint>
+    <link name="${name}_link" />
+    <joint name="${name}_joint" type="fixed">
+      <origin xyz="0 0 0" rpy="0 0 ${M_PI/2}" />
+      <parent link="${name}_center_link" />
       <child link="${name}_link" />
     </joint>

Commit message: fixed IMU orientation

File: panther_description/urdf/imu.urdf.xacro (robot description, xacro)
@@ -51,5 +51,5 @@
     <link name="${name}_link" />
     <joint name="${name}_joint" type="fixed">
-      <origin xyz="0 0 0" rpy="0 0 ${M_PI/2}" />
+      <origin xyz="0 0 0" rpy="0 0 ${-M_PI/2}" />
       <parent link="${name}_center_link" />
       <child link="${name}_link" />

Commit message: Fixed imu configuration

File: panther_description/urdf/imu.urdf.xacro (robot description, xacro)
@@ -26,6 +26,6 @@
 -->
 <robot xmlns:xacro="http://ros.org/wiki/xacro" name="imu">
-  <xacro:macro name="imu" params="name parent *joint_pose">
-    <link name="${name}_center_link">
+  <xacro:macro name="imu" params="parent *joint_pose">
+    <link name="imu_board_link">
       <inertial>
         <origin xyz="0.0002 0.003 -0.00025" rpy="0 0 0" />
@@ -44,14 +44,15 @@
       </visual>
     </link>
-    <joint name="${name}_center_joint" type="fixed">
+    <joint name="imu_board_joint" type="fixed">
       <xacro:insert_block name="joint_pose"/>
       <parent link="${parent}" />
-      <child link="${name}_center_link" />
+      <child link="imu_board_link" />
     </joint>
-    <link name="${name}_link" />
-    <joint name="${name}_joint" type="fixed">
-      <origin xyz="0 0 0" rpy="0 0 ${-M_PI/2}" />
-      <parent link="${name}_center_link" />
-      <child link="${name}_link" />
+    <!-- Required "base_imu_link" to read the razor IMU data -->
+    <link name="base_imu_link" />
+    <joint name="base_imu_joint" type="fixed">
+      <origin xyz="0 0 0" rpy="0 ${-M_PI/2} 0" />
+      <parent link="imu_board_link" />
+      <child link="base_imu_link" />
     </joint>
  </xacro:macro>

File: panther_description/urdf/panther.urdf.xacro (robot description, xacro)
@@ -75,5 +75,5 @@
   <!-- ZED - END -->
   <!-- IMU -->
-  <xacro:imu name="base_imu" parent="frame_link">
+  <xacro:imu parent="frame_link">
     <origin xyz="-0.0420817256507905 0 0.091441320597534" rpy="0 ${M_PI/2} 0" />
   </xacro:imu>
