Commit message: Added IMU and fixed TF reference

File: panther_description/urdf/chassis.urdf.xacro (robot description, xacro)
@@ -135,30 +135,4 @@
     <axis xyz="0 0 0" />
   </joint>
-  <link name="IMU_link">
-    <inertial>
-      <origin
-        xyz="0.002192 0.001241 0.000301"
-        rpy="0 0 0" />
-      <mass value="0.00456597126352491" />
-      <inertia ixx="2.67621227004883E-07" ixy="2.98461528217097E-08" ixz="2.61743631414246E-08"
-        iyy="9.30031615735385E-07" iyz="3.86352794956382E-09"
-        izz="6.80030175979387E-07" />
-    </inertial>
-    <visual>
-      <origin xyz="0 0 0" rpy="0 0 0" />
-      <geometry>
-        <mesh filename="${path_meshes}/chassis/IMU_link.STL" />
-      </geometry>
-      <material name="Red" />
-    </visual>
-  </link>
-  <joint name="IMU_joint" type="fixed">
-    <origin
-      xyz="0.0420817256507905 0 0.091441320597534"
-      rpy="3.13677140039975 -6.09351154012223E-17 -1.5707963267949" />
-    <parent link="frame_link" />
-    <child link="IMU_link" />
-    <axis xyz="0 0 0" />
-  </joint>
   <link name="connectors_link">
     <inertial>

File: panther_description/urdf/panther.urdf.xacro (robot description, xacro)
@@ -8,4 +8,5 @@
   <xacro:include filename="$(find panther_description)/urdf/gear.urdf.xacro" />
   <xacro:include filename="$(find panther_description)/urdf/zedcamera.urdf.xacro" />
+  <xacro:include filename="$(find panther_description)/urdf/imu.urdf.xacro" />
   <!-- Included URDF/XACRO Files -->
   <!-- Global properties -->
@@ -43,4 +44,9 @@
   </xacro:zedcamera>
   <!-- ZED - END -->
+  <!-- IMU -->
+  <xacro:imu name="base_imu" parent="frame_link">
+    <origin xyz="0.0420817256507905 0 0.091441320597534" rpy="${M_PI} ${M_PI/2} 0" />
+  </xacro:imu>
+  <!-- IMU -->
   <!-- Track -->
   <!-- passive_wheel_type tye: (1) continuous or (2) fixed -->
