Commit message: improved urdf

File: panther_description/urdf/chassis.urdf.xacro (robot description, xacro)
@@ -11,5 +11,5 @@
     </inertial>
     <visual>
-      <origin xyz="0 0 0" rpy="0 0 0" />
+      <origin xyz="0 0 0" rpy="0 0 ${M_PI}" />
       <geometry>
         <mesh filename="${path_meshes}/chassis/frame_link.STL" />
@@ -33,5 +33,5 @@
     </inertial>
     <visual>
-      <origin xyz="0 0 0" rpy="0 0 0" />
+      <origin xyz="0 0 0" rpy="0 0 ${M_PI}" />
       <geometry>
         <mesh filename="${path_meshes}/chassis/iron_link.STL" />
@@ -55,5 +55,5 @@
     </inertial>
     <visual>
-      <origin xyz="0 0 0" rpy="0 0 0" />
+      <origin xyz="0 0 0" rpy="0 0 ${M_PI}" />
       <geometry>
         <mesh filename="${path_meshes}/chassis/cover_link.STL" />
@@ -78,5 +78,5 @@
     </inertial>
     <visual>
-      <origin xyz="0 0 0" rpy="0 0 0" />
+      <origin xyz="0 0 0" rpy="0 0 ${M_PI}" />
       <geometry>
         <mesh filename="${path_meshes}/chassis/antenna_link.STL" />
@@ -100,5 +100,5 @@
     </inertial>
     <visual>
-      <origin xyz="0 0 0" rpy="0 0 0" />
+      <origin xyz="0 0 0" rpy="0 0 ${M_PI}" />
       <geometry>
         <mesh filename="${path_meshes}/chassis/speaker_link.STL" />
@@ -115,5 +115,5 @@
   <link name="charge_Link">
     <inertial>
-      <origin xyz="-0.00065 0.0040 0.00065" rpy="0 0 0" />
+      <origin xyz="-0.00065 0.0040 0.00065" rpy="0 0 ${M_PI}" />
       <mass value="0.0049" />
       <inertia ixx="1.88298361729241E-07" ixy="-9.05119559629111E-09" ixz="1.84328236191772E-09"
@@ -122,5 +122,5 @@
     </inertial>
     <visual>
-      <origin xyz="0 0 0" rpy="0 0 0" />
+      <origin xyz="0 0 0" rpy="0 0 ${M_PI}" />
       <geometry>
         <mesh filename="${path_meshes}/chassis/charge_link.STL" />
@@ -144,5 +144,5 @@
     </inertial>
     <visual>
-      <origin xyz="0 0 0" rpy="0 0 0" />
+      <origin xyz="0 0 0" rpy="0 0 ${M_PI}" />
       <geometry>
         <mesh filename="${path_meshes}/chassis/connectors_link.STL" />
@@ -175,6 +175,6 @@
   <joint name="ssd_joint" type="fixed">
     <origin
-      xyz="-0.0465581999999993 0.0307500000000006 0.0467424000000017"
-      rpy="3.14159265358979 0 0" />
+      xyz="0.0465 0.03075 0.04674"
+      rpy="${M_PI} 0 ${M_PI}" />
     <parent link="frame_link" />
     <child link="ssd_link" />
@@ -199,6 +199,6 @@
   <joint name="jetson_carrier_joint" type="fixed">
     <origin
-      xyz="-0.1 0.01 0.055"
-      rpy="-1.5707963267949 0 0" />
+      xyz="0.1 0.01 0.055"
+      rpy="${-M_PI/2} 0 ${M_PI}" />
     <parent link="frame_link" />
     <child link="jetson_carrier_link" />
@@ -245,5 +245,5 @@
   </link>
   <joint name="battery_joint" type="fixed">
-    <origin xyz="0.13 0 0.01" rpy="0 0 0" />
+    <origin xyz="-0.13 0 0.01" rpy="0 0 0" />
     <parent link="frame_link" />
     <child link="battery_link" />
@@ -260,5 +260,5 @@
   </link>
   <joint name="unav_joint" type="fixed">
-    <origin xyz="0.10 0 0.13" rpy="0 0 0" />
+    <origin xyz="-0.10 0 0.13" rpy="0 0 0" />
     <parent link="frame_link" />
     <child link="unav_link" />

File: panther_description/urdf/gear.urdf.xacro (robot description, xacro)
@@ -1,6 +1,6 @@
 <?xml version="1.0"?>
 <robot xmlns:xacro="http://ros.org/wiki/xacro" name="gear">
- <xacro:macro name="gear" params="position parent *joint_pose">
-  <link name="gear_${position}_Link">
+ <xacro:macro name="gear" params="type orientation">
+  <link name="gear_${type}_Link">
     <inertial>
       <origin xyz="0 0 0.008" rpy="0 ${M_PI} 0" />
@@ -18,11 +18,13 @@
     </visual>
   </link>
-  <joint name="gear_${position}_joint" type="continuous">
-    <xacro:insert_block name="joint_pose"/>
-    <parent link="track_${position}_link" />
-    <child link="gear_${position}_Link" />
-    <axis xyz="0 0 -1" />
+  <joint name="gear_${type}_joint" type="continuous">
+    <origin
+      xyz="-0.0536535102814494 -0.00979339452125411 0.0186240655062149"
+      rpy="-${M_PI/2} ${M_PI} ${M_PI}" />
+    <parent link="track_${type}_link" />
+    <child link="gear_${type}_Link" />
+    <axis xyz="0 0 ${-1 * orientation}" />
     <!-- Passive sprocket rotate automatically according to the status of the active one -->
-    <mimic joint="${position}_joint" multiplier="${sprocket_teeth/gear_teeth}" offset="0"/>
+    <mimic joint="${type}_joint" multiplier="${sprocket_teeth/gear_teeth}" offset="0"/>
   </joint>
   </xacro:macro>

File: panther_description/urdf/panther.urdf.xacro (robot description, xacro)
@@ -28,10 +28,8 @@
   <!-- Included URDF/XACRO Files -->
   <xacro:include filename="$(find panther_description)/urdf/materials.urdf" />
+  <xacro:include filename="$(find panther_description)/urdf/chassis.urdf.xacro" />
   <xacro:include filename="$(find panther_description)/urdf/track.urdf.xacro" />
-  <xacro:include filename="$(find panther_description)/urdf/chassis.urdf.xacro" />
-  <xacro:include filename="$(find panther_description)/urdf/sprocket.urdf.xacro" />
-  <xacro:include filename="$(find panther_description)/urdf/gear.urdf.xacro" />
-  <xacro:include filename="$(find panther_description)/urdf/zedcamera.urdf.xacro" />
-  <xacro:include filename="$(find panther_description)/urdf/imu.urdf.xacro" />
+  <!--<xacro:include filename="$(find panther_description)/urdf/zedcamera.urdf.xacro" />
+  <xacro:include filename="$(find panther_description)/urdf/imu.urdf.xacro" />-->
   <!-- Included URDF/XACRO Files -->
   <!-- Global properties -->
@@ -58,5 +56,5 @@
                                izz="1" />
     </inertial>
-    <visual>
+    <!--<visual>
       <origin xyz="0 0 0" rpy="0 0 0" />
       <geometry>
@@ -64,9 +62,9 @@
       </geometry>
       <material name="Green" />
-    </visual>
+    </visual>-->
   </link>
   <!-- Chassis -->
   <xacro:chassis parent="base_link">
-    <origin xyz="0 0 0.08" rpy="0 0 3.14159" />
+    <origin xyz="0 0 0.08" rpy="0 0 0" />
   </xacro:chassis>
   <!-- Chassis - END -->
@@ -82,27 +80,6 @@
   <!-- IMU -->
   <!-- Track -->
-  <!-- passive_wheel_type type: (1) continuous or (2) fixed -->
-  <xacro:track position="left" parent="frame_link" passive_wheel_type="continuous">
-    <origin
-      xyz="0 -0.161 -0.014"
-      rpy="0 0 0" />
-    <origin
-      xyz="0.15476 -0.161 ${-0.014 - 0.0267}"
-      rpy="-${M_PI/2} 0 0" />
-    <origin
-      xyz="0.054 -0.010 0.019"
-      rpy="-${M_PI/2} 0 0" />
-  </xacro:track>
-  <xacro:track position="right" parent="frame_link" passive_wheel_type="continuous">
-    <origin
-      xyz="0 0.161 -0.014"
-      rpy="0 0 0" />
-    <origin
-      xyz="0.155 0.161 ${-0.014 - 0.0267}"
-      rpy="-${M_PI/2} 0 0" />
-    <origin
-      xyz="0.054 0.010 0.019"
-      rpy="${M_PI/2} 0 0" />
-  </xacro:track>
+  <xacro:track type="left" parent="frame_link" />
+  <xacro:track type="right" parent="frame_link" />
   <!-- Track - END -->
   </xacro:macro>

File: panther_description/urdf/track.urdf.xacro (robot description, xacro)
@@ -26,149 +26,158 @@
 -->
 <robot xmlns:xacro="http://ros.org/wiki/xacro" name="track">
- <!-- passive_wheel_type tye: (1) continuous or (2) fixed -->
- <xacro:macro name="track" params="position parent passive_wheel_type *track_pose *joint_pose *gear_pose">
+  <xacro:include filename="$(find panther_description)/urdf/sprocket.urdf.xacro" />
+  <xacro:include filename="$(find panther_description)/urdf/gear.urdf.xacro" />
+  <xacro:include filename="$(find panther_description)/urdf/wheel.urdf.xacro" />
+  <xacro:macro name="track" params="type parent">
+  <!-- Define orientation -->
+  <xacro:if value="${type == 'left'}">
+    <xacro:property name="orientation" value="-1"/>
+  </xacro:if>
+  <xacro:if value="${type == 'right'}">
+    <xacro:property name="orientation" value="1"/>
+  </xacro:if>
   <!-- TRACK FIXED LINKS -->
-  <link name="track_${position}_link">
+  <link name="track_${type}_link">
     <inertial>
       <origin xyz="-0.0168 0.0080 0.0061" rpy="0 0 0" />
       <mass value="0.512" />
-      <inertia ixx="0.0008" ixy="0" ixz="0"
-        iyy="0.005" iyz="0.0001"
-        izz="0.005" />
-    </inertial>
-    <visual>
-      <origin xyz="0 0 0" rpy="0 0 0" />
-      <geometry>
-        <mesh filename="${path_meshes}/track/${position}/track_link.STL" />
+      <inertia ixx="0.0008" ixy="0"     ixz="0"
+                            iyy="0.005" iyz="0.0001"
+                                        izz="0.005" />
+    </inertial>
+    <visual>
+      <origin xyz="0 0 0" rpy="0 0 ${M_PI}" />
+      <geometry>
+        <mesh filename="${path_meshes}/track/${type}/track_link.STL" />
       </geometry>
       <material name="White-Alpha" />
     </visual>
   </link>
-  <joint name="track_${position}_joint" type="fixed">
-    <xacro:insert_block name="track_pose"/>
+  <joint name="track_${type}_joint" type="fixed">
+    <origin xyz="0 ${orientation * -0.161} -0.014" rpy="0 0 0" />
     <parent link="${parent}" />
-    <child link="track_${position}_link" />
-    <axis xyz="0 0 0" />
-  </joint>
-  <link name="iron_${position}_Link">
+    <child link="track_${type}_link" />
+    <axis xyz="0 0 0" />
+  </joint>
+  <link name="iron_${type}_Link">
     <inertial>
       <origin xyz="0.028 0.026 0.011" rpy="0 0 0" />
       <mass value="1.412" />
       <inertia ixx="0.0021" ixy="0.0009" ixz="0.0003"
-        iyy="0.0080" iyz="0.0002"
-        izz="0.009" />
-    </inertial>
-    <visual>
-      <origin xyz="0 0 0" rpy="0 0 0" />
-      <geometry>
-        <mesh filename="${path_meshes}/track/${position}/iron_link.STL" />
+                            iyy="0.0080" iyz="0.0002"
+                                         izz="0.009" />
+    </inertial>
+    <visual>
+      <origin xyz="0 0 0" rpy="0 0 ${M_PI}" />
+      <geometry>
+        <mesh filename="${path_meshes}/track/${type}/iron_link.STL" />
       </geometry>
       <material name="GunMetalGrey" />
     </visual>
   </link>
-  <joint name="iron_${position}_joint" type="fixed">
-    <origin xyz="0 0 0" rpy="0 0 0" />
-    <parent link="track_${position}_link" />
-    <child link="iron_${position}_Link" />
-    <axis xyz="0 0 0" />
-  </joint>
-  <link name="damper_${position}_Link">
+  <joint name="iron_${type}_joint" type="fixed">
+    <origin xyz="0 0 0" rpy="0 0 0" />
+    <parent link="track_${type}_link" />
+    <child link="iron_${type}_Link" />
+    <axis xyz="0 0 0" />
+  </joint>
+  <link name="damper_${type}_Link">
     <inertial>
       <origin xyz="0.011 0.014 0.028" rpy="0 0 0" />
       <mass value="0.028" />
-      <inertia ixx="0" ixy="0" ixz="0"
-        iyy="0.0007" iyz="0"
-        izz="0.0002" />
-    </inertial>
-    <visual>
-      <origin xyz="0 0 0" rpy="0 0 0" />
-      <geometry>
-        <mesh filename="${path_meshes}/track/${position}/damper_link.STL" />
+      <inertia ixx="0" ixy="0"      ixz="0"
+                       iyy="0.0007" iyz="0"
+                                    izz="0.0002" />
+    </inertial>
+    <visual>
+      <origin xyz="0 0 0" rpy="0 0 ${M_PI}" />
+      <geometry>
+        <mesh filename="${path_meshes}/track/${type}/damper_link.STL" />
       </geometry>
       <material name="Black" />
     </visual>
   </link>
-  <joint name="damper_${position}_joint" type="fixed">
-    <origin xyz="0 0 0" rpy="0 0 0" />
-    <parent link="track_${position}_link" />
-    <child link="damper_${position}_Link" />
-    <axis xyz="0 0 0" />
-  </joint>
-  <link name="damper_label_${position}_Link">
+  <joint name="damper_${type}_joint" type="fixed">
+    <origin xyz="0 0 0" rpy="0 0 0" />
+    <parent link="track_${type}_link" />
+    <child link="damper_${type}_Link" />
+    <axis xyz="0 0 0" />
+  </joint>
+  <link name="damper_label_${type}_Link">
     <inertial>
       <origin xyz="0.0111 0.0137 0.0341" rpy="0 0 0" />
       <mass value="0.0062" />
       <inertia ixx="0" ixy="0" ixz="0"
-        iyy="0" iyz="0"
-        izz="0" />
-    </inertial>
-    <visual>
-      <origin xyz="0 0 0" rpy="0 0 0" />
-      <geometry>
-        <mesh filename="${path_meshes}/track/${position}/damper_label_link.STL" />
+                       iyy="0" iyz="0"
+                               izz="0" />
+    </inertial>
+    <visual>
+      <origin xyz="0 0 0" rpy="0 0 ${M_PI}" />
+      <geometry>
+        <mesh filename="${path_meshes}/track/${type}/damper_label_link.STL" />
       </geometry>
       <material name="Pink" />
     </visual>
   </link>
-  <joint name="damper_label_${position}_joint" type="fixed">
-    <origin xyz="0 0 0" rpy="0 0 0" />
-    <parent link="damper_${position}_Link" />
-    <child link="damper_label_${position}_Link" />
-    <axis xyz="0 0 0" />
-  </joint>
-  <link name="fender_${position}_Link">
+  <joint name="damper_label_${type}_joint" type="fixed">
+    <origin xyz="0 0 0" rpy="0 0 0" />
+    <parent link="damper_${type}_Link" />
+    <child link="damper_label_${type}_Link" />
+    <axis xyz="0 0 0" />
+  </joint>
+  <link name="fender_${type}_Link">
     <inertial>
       <origin xyz="-0.0044 0.0167 0.0872" rpy="0 0 0" />
       <mass value="0.0853" />
-      <inertia ixx="0" ixy="0" ixz="0"
-        iyy="0.0007" iyz="0"
-        izz="0.0007" />
-    </inertial>
-    <visual>
-      <origin xyz="0 0 0" rpy="0 0 0" />
-      <geometry>
-        <mesh filename="${path_meshes}/track/${position}/fender_link.STL" />
+      <inertia ixx="0" ixy="0"      ixz="0"
+                       iyy="0.0007" iyz="0"
+                                    izz="0.0007" />
+    </inertial>
+    <visual>
+      <origin xyz="0 0 0" rpy="0 0 ${M_PI}" />
+      <geometry>
+        <mesh filename="${path_meshes}/track/${type}/fender_link.STL" />
       </geometry>
       <material name="Black" />
     </visual>
   </link>
-  <joint name="fender_${position}_joint" type="fixed">
-    <origin xyz="0 0 0" rpy="0 0 0" />
-    <parent link="track_${position}_link" />
-    <child link="fender_${position}_Link" />
-    <axis xyz="0 0 0" />
-  </joint>
-  <link name="chain_${position}_Link">
+  <joint name="fender_${type}_joint" type="fixed">
+    <origin xyz="0 0 0" rpy="0 0 0" />
+    <parent link="track_${type}_link" />
+    <child link="fender_${type}_Link" />
+    <axis xyz="0 0 0" />
+  </joint>
+  <link name="chain_${type}_Link">
     <inertial>
       <origin xyz="0.101 0.0001 -0.0026" rpy="0 0 0" />
       <mass value="0.0708" />
       <inertia ixx="0" ixy="0" ixz="0"
-        iyy="0" iyz="0"
-        izz="0.0001" />
-    </inertial>
-    <visual>
-      <origin xyz="0 0 0" rpy="0 0 0" />
-      <geometry>
-        <mesh filename="${path_meshes}/track/${position}/chain_link.STL" />
+                       iyy="0" iyz="0"
+                               izz="0.0001" />
+    </inertial>
+    <visual>
+      <origin xyz="0 0 0" rpy="0 0 ${M_PI}" />
+      <geometry>
+        <mesh filename="${path_meshes}/track/${type}/chain_link.STL" />
       </geometry>
       <material name="DarkGrey" />
     </visual>
   </link>
-  <joint name="chain_${position}_joint" type="fixed">
-    <origin xyz="0 0 0" rpy="0 0 0" />
-    <parent link="track_${position}_link" />
-    <child link="chain_${position}_Link" />
-    <axis xyz="0 0 0" />
-  </joint>
-  <link name="rubber_${position}_Link">
+  <joint name="chain_${type}_joint" type="fixed">
+    <origin xyz="0 0 0" rpy="0 0 0" />
+    <parent link="track_${type}_link" />
+    <child link="chain_${type}_Link" />
+    <axis xyz="0 0 0" />
+  </joint>
+  <link name="rubber_${type}_Link">
     <inertial>
       <origin xyz="-0.0137 0 -0.0014" rpy="0 0 0" />
       <mass value="0.466" />
-      <inertia ixx="0.0016" ixy="0" ixz="-0.0003"
-        iyy="0.0090" iyz="0"
-        izz="0.007" />
-    </inertial>
-    <visual>
-      <origin xyz="0 0 0" rpy="0 0 0" />
+      <inertia ixx="0.0016" ixy="0"      ixz="-0.0003"
+                            iyy="0.0090" iyz="0"
+                                         izz="0.007" />
+    </inertial>
+    <visual>
+      <origin xyz="0 0 0" rpy="0 0 ${M_PI}" />
       <geometry>
         <mesh filename="${path_meshes}/track/rubber_link.STL" />
@@ -177,226 +186,85 @@
     </visual>
   </link>
-  <joint name="rubber_${position}_joint" type="fixed">
-    <origin xyz="0 0 0" rpy="0 0 0" />
-    <parent link="track_${position}_link" />
-    <child link="rubber_${position}_Link" />
+  <joint name="rubber_${type}_joint" type="fixed">
+    <origin xyz="0 0 0" rpy="0 0 0" />
+    <parent link="track_${type}_link" />
+    <child link="rubber_${type}_Link" />
     <axis xyz="0 0 0" />
   </joint>
   <!-- Sprocket -->
-  <xacro:sprocket position="${position}" parent="${parent}">
-    <xacro:insert_block name="joint_pose"/>
-  </xacro:sprocket>
-  <!-- Sprocket - END -->
+  <xacro:sprocket type="${type}" orientation="${orientation}" parent="${parent}" />
   <!-- Gear -->
-  <xacro:gear position="${position}" parent="track_${position}_link">
-    <xacro:insert_block name="gear_pose"/>
-  </xacro:gear>
-  <!-- Gear - END -->
-  <!-- PASSIVE WHEELS -->
-  <link name="wheel_${position}_center_up_Link">
-    <inertial>
-      <origin xyz="0 0 0" rpy="0 0 0" />
-      <mass value="0.016" />
-      <inertia ixx="0" ixy="0" ixz="0"
-                       iyy="0" iyz="0"
-                               izz="0" />
-    </inertial>
-    <visual>
-      <origin xyz="0 0 0" rpy="0 0 0" />
-      <geometry>
-        <mesh filename="${path_meshes}/track/wheel_center_up_link.STL" />
-      </geometry>
-      <material name="White-Alpha" />
-    </visual>
-  </link>
-  <joint name="wheel_${position}_center_up_joint" type="${passive_wheel_type}">
-    <origin
-      xyz="0 0 0.0735790044064745"
-      rpy="-${M_PI/2} 0 0" />
-    <parent link="track_${position}_link" />
-    <child link="wheel_${position}_center_up_Link" />
-    <axis xyz="0 0 -1" />
-    <xacro:if value="${passive_wheel_type == 'continuous'}">
-    <!-- Passive sprocket rotate automatically according to the status of the active one -->
-      <mimic joint="${position}_joint" multiplier="1" offset="0"/>
-    </xacro:if>
-  </joint>
-  <link name="wheel_${position}_front_up_Link">
-    <inertial>
+  <xacro:gear type="${type}" orientation="${orientation}" />
+  <!-- Passive wheels -->
+  <xacro:wheel type="${type}" orientation="${orientation}" conf="front_down" name="wheel_front_link" passive_wheel_type="continuous">
+      <!-- visual wheel origin offest-->
       <origin xyz="0 0 0.020143" rpy="0 0 0" />
-      <mass value="0.043" />
-      <inertia ixx="0" ixy="0" ixz="0"
-                       iyy="0" iyz="0"
-                               izz="0" />
-    </inertial>
-    <visual>
+      <!-- joint origin -->
+      <origin
+        xyz="0.157 0 -0.034"
+        rpy="${orientation * M_PI/2} 0 0" />
+      <!-- collisione shape -->
+      <cylinder length="0.05" radius="0.025"/>
+  </xacro:wheel>
+  <xacro:wheel type="${type}" orientation="${orientation}" conf="front_up" name="wheel_front_link" passive_wheel_type="continuous">
+      <!-- visual wheel origin offest-->
       <origin xyz="0 0 0.020143" rpy="0 0 0" />
-      <geometry>
-        <mesh filename="${path_meshes}/track/wheel_front_link.STL" />
-      </geometry>
-      <material name="White-Alpha" />
-    </visual>
-  </link>
-  <joint name="wheel_${position}_front_up_joint" type="${passive_wheel_type}">
-    <origin
-      xyz="-0.18867 0 0.010536"
-      rpy="-${M_PI/2} 0 0" />
-    <parent link="track_${position}_link" />
-    <child link="wheel_${position}_front_up_Link" />
-    <axis xyz="0 0 -1" />
-    <xacro:if value="${passive_wheel_type == 'continuous'}">
-    <!-- Passive sprocket rotate automatically according to the status of the active one -->
-      <mimic joint="${position}_joint" multiplier="1" offset="0"/>
-    </xacro:if>
-  </joint>
-  <!-- Front passive wheel all time type continous -->
-  <link name="wheel_${position}_front_down_Link">
-    <inertial>
-      <origin xyz="0 0 0.020143" rpy="0 0 0" />
-      <mass value="0.0431" />
-      <inertia ixx="0" ixy="0" ixz="0"
-                       iyy="0" iyz="0"
-                               izz="0" />
-    </inertial>
-    <visual>
-      <origin xyz="0 0 0.020143" rpy="0 0 0" />
-      <geometry>
-        <mesh filename="${path_meshes}/track/wheel_front_link.STL" />
-      </geometry>
-      <material name="White-Alpha" />
-    </visual>
-    <collision>
-      <origin xyz="0 0 -0.025" rpy="0 0 0" />
-      <geometry>
-        <cylinder length="0.05" radius="0.025"/>
-      </geometry>
-    </collision>
-  </link>
-  <joint name="wheel_${position}_front_down_joint" type="${passive_wheel_type}">
-    <origin
-      xyz="-0.15659 0 -0.034143"
-      rpy="-${M_PI/2} 0 0" />
-    <parent link="track_${position}_link" />
-    <child link="wheel_${position}_front_down_Link" />
-    <axis xyz="0 0 -1" />
-    <xacro:if value="${passive_wheel_type == 'continuous'}">
-    <!-- Passive sprocket rotate automatically according to the status of the active one -->
-      <mimic joint="${position}_joint" multiplier="1" offset="0"/>
-    </xacro:if>
-  </joint>
-  <link name="wheel_${position}_center_A_Link">
-    <inertial>
-      <origin xyz="-0.064 -0.046 0.004" rpy="0 0 0" />
-      <mass value="0.0082" />
-      <inertia ixx="0" ixy="0" ixz="0"
-                       iyy="0" iyz="0"
-                               izz="0" />
-    </inertial>
-    <visual>
-      <origin xyz="0 0 0" rpy="0 0 0" />
-      <geometry>
-        <mesh filename="${path_meshes}/track/wheel_center_link.STL" />
-      </geometry>
-      <material name="White-Alpha" />
-    </visual>
-  </link>
-  <joint name="wheel_${position}_center_A_joint" type="${passive_wheel_type}">
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