Commit message: improved urdf

File: panther_description/urdf/wheel.urdf.xacro (robot description, xacro)
@@ -25,52 +25,39 @@
 EVEN IF ADVISED OF THE POSSIBILITY OF SUCH DAMAGE.
 -->
-<robot xmlns:xacro="http://ros.org/wiki/xacro" name="sprocket">
- <xacro:macro name="sprocket" params="type orientation parent">
-  <link name="sprocket_${type}_Link">
+<robot xmlns:xacro="http://ros.org/wiki/xacro" name="wheel">
+  <xacro:macro name="wheel" params="type orientation conf name passive_wheel_type *visual_pose *wheel_pose *collision_shape">
+  <!-- Front passive wheel all time type continous -->
+  <link name="wheel_${type}_${conf}_Link">
     <inertial>
-      <origin xyz="0 0 0" rpy="0 0 0" />
-      <mass value="0.098" />
-      <inertia ixx="1" ixy="0" ixz="0"
-                       iyy="1" iyz="0"
-                               izz="1" />
+      <origin xyz="0 0 0.020143" rpy="0 0 0" />
+      <mass value="0.0431" />
+      <inertia ixx="0" ixy="0" ixz="0"
+                       iyy="0" iyz="0"
+                               izz="0" />
     </inertial>
-    <!-- Visual mesh -->
     <visual>
-      <origin
-        xyz="0 0 ${sprocket_leght / 2 - 0.005}"
-        rpy="0 0 0" />
+      <xacro:insert_block name="visual_pose"/>
       <geometry>
-        <mesh filename="${path_meshes}/track/sprocket_link.STL" />
+        <mesh filename="${path_meshes}/track/${name}.STL" />
       </geometry>
-      <material name="Black" />
+      <material name="White-Alpha" />
     </visual>
-    <!-- Collision cylinder -->
     <collision>
       <origin xyz="0 0 0" rpy="0 0 0" />
       <geometry>
-        <cylinder length="${sprocket_leght}" radius="${sprocket_radius}"/>
+        <xacro:insert_block name="collision_shape"/>
       </geometry>
-      <material name="Red" />
     </collision>
   </link>
-  <!-- Joint properties -->
-  <joint name="${type}_joint" type="continuous">
-    <origin xyz="-0.15476 ${orientation * -0.161} ${-0.014 - 0.0267}" rpy="${orientation * M_PI/2} 0 0" />
-    <parent link="${parent}" />
-    <child link="sprocket_${type}_Link" />
+  <joint name="wheel_${type}_${conf}_joint" type="${passive_wheel_type}">
+    <xacro:insert_block name="wheel_pose"/>
+    <parent link="track_${type}_link" />
+    <child link="wheel_${type}_${conf}_Link" />
     <axis xyz="0 0 ${-1 * orientation}" />
-    <limit effort="12" velocity="22"/>
-    <joint_properties damping="1.0" friction="1.0"/>
+    <!-- Passive sprocket rotate automatically according to the status of the active one -->
+    <xacro:if value="${passive_wheel_type == 'continuous'}">
+      <mimic joint="${type}_joint" multiplier="1" offset="0"/>
+    </xacro:if>
   </joint>
-  <!-- Transmission -->
-  <transmission name="${type}_trans" type="SimpleTransmission">
-    <type>transmission_interface/SimpleTransmission</type>
-    <actuator name="${type}_motor">
-      <mechanicalReduction>${gear_teeth/sprocket_teeth}</mechanicalReduction>
-    </actuator>
-    <joint name="${type}_joint">
-      <hardwareInterface>hardware_interface/VelocityJointInterface</hardwareInterface>
-    </joint>
-  </transmission>
   </xacro:macro>
 </robot>

Commit message: Added license and fixed some other errors

File: panther_description/urdf/chassis.urdf.xacro (robot description, xacro)
@@ -1,3 +1,28 @@
 <?xml version="1.0"?>
+<!--
+Copyright (C) 2017, Raffaello Bonghi <raffaello@rnext.it>
+All rights reserved
+Redistribution and use in source and binary forms, with or without
+modification, are permitted provided that the following conditions are met:
+1. Redistributions of source code must retain the above copyright
+   notice, this list of conditions and the following disclaimer.
+2. Redistributions in binary form must reproduce the above copyright
+   notice, this list of conditions and the following disclaimer in the
+   documentation and/or other materials provided with the distribution.
+3. Neither the name of the copyright holder nor the names of its
+   contributors may be used to endorse or promote products derived
+   from this software without specific prior written permission.
+THIS SOFTWARE IS PROVIDED BY THE COPYRIGHT HOLDERS AND
+CONTRIBUTORS "AS IS" AND ANY EXPRESS OR IMPLIED WARRANTIES, INCLUDING,
+BUT NOT LIMITED TO, THE IMPLIED WARRANTIES OF MERCHANTABILITY AND FITNESS
+FOR A PARTICULAR PURPOSE ARE DISCLAIMED. IN NO EVENT SHALL THE COPYRIGHT
+HOLDER OR CONTRIBUTORS BE LIABLE FOR ANY DIRECT, INDIRECT, INCIDENTAL,
+SPECIAL, EXEMPLARY, OR CONSEQUENTIAL DAMAGES (INCLUDING, BUT NOT LIMITED TO,
+PROCUREMENT OF SUBSTITUTE GOODS OR SERVICES; LOSS OF USE, DATA, OR PROFITS;
+OR BUSINESS INTERRUPTION) HOWEVER CAUSED AND ON ANY THEORY OF LIABILITY,
+WHETHER IN CONTRACT, STRICT LIABILITY, OR TORT (INCLUDING NEGLIGENCE
+OR OTHERWISE) ARISING IN ANY WAY OUT OF THE USE OF THIS SOFTWARE,
+EVEN IF ADVISED OF THE POSSIBILITY OF SUCH DAMAGE.
+-->
 <robot xmlns:xacro="http://ros.org/wiki/xacro" name="chassis">
   <xacro:macro name="chassis" params="parent *joint_pose">
@@ -17,4 +42,11 @@
       <material name="Black" />
     </visual>
+    <collision>
+      <origin xyz="0 0 0.09" rpy="0 0 0" />
+      <geometry>
+        <box size="0.42 0.26 0.18" />
+      </geometry>
+      <material name="Red" />
+    </collision>
   </link>
   <joint name="frame_joint" type="fixed">

File: panther_description/urdf/description.xacro (robot description, xacro)
@@ -1,23 +1,27 @@
 <?xml version="1.0"?>
 <!--
-Software License Agreement (BSD)
-\file      description.urdf.xacro
-\authors   Raffaello Bonghi <raffaello@rnext.it
-\copyright Copyright (c) 2016, Raffaello Bonghi, All rights reserved.
-Redistribution and use in source and binary forms, with or without modification, are permitted provided that
-the following conditions are met:
- * Redistributions of source code must retain the above copyright notice, this list of conditions and the
-   following disclaimer.
- * Redistributions in binary form must reproduce the above copyright notice, this list of conditions and the
-   following disclaimer in the documentation and/or other materials provided with the distribution.
- * Neither the name of Clearpath Robotics nor the names of its contributors may be used to endorse or promote
-   products derived from this software without specific prior written permission.
-THIS SOFTWARE IS PROVIDED BY THE COPYRIGHT HOLDERS AND CONTRIBUTORS "AS IS" AND ANY EXPRESS OR IMPLIED WAR-
-RANTIES, INCLUDING, BUT NOT LIMITED TO, THE IMPLIED WARRANTIES OF MERCHANTABILITY AND FITNESS FOR A PARTICULAR
-PURPOSE ARE DISCLAIMED. IN NO EVENT SHALL THE COPYRIGHT HOLDER OR CONTRIBUTORS BE LIABLE FOR ANY DIRECT, IN-
-DIRECT, INCIDENTAL, SPECIAL, EXEMPLARY, OR CONSEQUENTIAL DAMAGES (INCLUDING, BUT NOT LIMITED TO, PROCUREMENT
-OF SUBSTITUTE GOODS OR SERVICES; LOSS OF USE, DATA, OR PROFITS; OR BUSINESS INTERRUPTION) HOWEVER CAUSED AND
-ON ANY THEORY OF LIABILITY, WHETHER IN CONTRACT, STRICT LIABILITY, OR TORT (INCLUDING NEGLIGENCE OR OTHERWISE)
-ARISING IN ANY WAY OUT OF THE USE OF THIS SOFTWARE, EVEN IF ADVISED OF THE POSSIBILITY OF SUCH DAMAGE.
+Copyright (C) 2017, Raffaello Bonghi <raffaello@rnext.it>
+All rights reserved
+Redistribution and use in source and binary forms, with or without
+modification, are permitted provided that the following conditions are met:
+1. Redistributions of source code must retain the above copyright
+   notice, this list of conditions and the following disclaimer.
+2. Redistributions in binary form must reproduce the above copyright
+   notice, this list of conditions and the following disclaimer in the
+   documentation and/or other materials provided with the distribution.
+3. Neither the name of the copyright holder nor the names of its
+   contributors may be used to endorse or promote products derived
+   from this software without specific prior written permission.
+THIS SOFTWARE IS PROVIDED BY THE COPYRIGHT HOLDERS AND
+CONTRIBUTORS "AS IS" AND ANY EXPRESS OR IMPLIED WARRANTIES, INCLUDING,
+BUT NOT LIMITED TO, THE IMPLIED WARRANTIES OF MERCHANTABILITY AND FITNESS
+FOR A PARTICULAR PURPOSE ARE DISCLAIMED. IN NO EVENT SHALL THE COPYRIGHT
+HOLDER OR CONTRIBUTORS BE LIABLE FOR ANY DIRECT, INDIRECT, INCIDENTAL,
+SPECIAL, EXEMPLARY, OR CONSEQUENTIAL DAMAGES (INCLUDING, BUT NOT LIMITED TO,
+PROCUREMENT OF SUBSTITUTE GOODS OR SERVICES; LOSS OF USE, DATA, OR PROFITS;
+OR BUSINESS INTERRUPTION) HOWEVER CAUSED AND ON ANY THEORY OF LIABILITY,
+WHETHER IN CONTRACT, STRICT LIABILITY, OR TORT (INCLUDING NEGLIGENCE
+OR OTHERWISE) ARISING IN ANY WAY OUT OF THE USE OF THIS SOFTWARE,
+EVEN IF ADVISED OF THE POSSIBILITY OF SUCH DAMAGE.
 -->
 <robot name="panther" xmlns:xacro="http://ros.org/wiki/xacro">

File: panther_description/urdf/gear.urdf.xacro (robot description, xacro)
@@ -42,4 +42,10 @@
       <material name="DarkGrey" />
     </visual>
+    <collision>
+      <origin xyz="0 0 0" rpy="0 0 0" />
+      <geometry>
+        <cylinder length="0.01" radius="0.016"/>
+      </geometry>
+    </collision>
   </link>
   <joint name="gear_${type}_joint" type="continuous">

File: panther_description/urdf/imu.urdf.xacro (robot description, xacro)
@@ -1,3 +1,28 @@
 <?xml version="1.0"?>
+<!--
+Copyright (C) 2017, Raffaello Bonghi <raffaello@rnext.it>
+All rights reserved
+Redistribution and use in source and binary forms, with or without
+modification, are permitted provided that the following conditions are met:
+1. Redistributions of source code must retain the above copyright
+   notice, this list of conditions and the following disclaimer.
+2. Redistributions in binary form must reproduce the above copyright
+   notice, this list of conditions and the following disclaimer in the
+   documentation and/or other materials provided with the distribution.
+3. Neither the name of the copyright holder nor the names of its
+   contributors may be used to endorse or promote products derived
+   from this software without specific prior written permission.
+THIS SOFTWARE IS PROVIDED BY THE COPYRIGHT HOLDERS AND
+CONTRIBUTORS "AS IS" AND ANY EXPRESS OR IMPLIED WARRANTIES, INCLUDING,
+BUT NOT LIMITED TO, THE IMPLIED WARRANTIES OF MERCHANTABILITY AND FITNESS
+FOR A PARTICULAR PURPOSE ARE DISCLAIMED. IN NO EVENT SHALL THE COPYRIGHT
+HOLDER OR CONTRIBUTORS BE LIABLE FOR ANY DIRECT, INDIRECT, INCIDENTAL,
+SPECIAL, EXEMPLARY, OR CONSEQUENTIAL DAMAGES (INCLUDING, BUT NOT LIMITED TO,
+PROCUREMENT OF SUBSTITUTE GOODS OR SERVICES; LOSS OF USE, DATA, OR PROFITS;
+OR BUSINESS INTERRUPTION) HOWEVER CAUSED AND ON ANY THEORY OF LIABILITY,
+WHETHER IN CONTRACT, STRICT LIABILITY, OR TORT (INCLUDING NEGLIGENCE
+OR OTHERWISE) ARISING IN ANY WAY OUT OF THE USE OF THIS SOFTWARE,
+EVEN IF ADVISED OF THE POSSIBILITY OF SUCH DAMAGE.
+-->
 <robot xmlns:xacro="http://ros.org/wiki/xacro" name="imu">
   <xacro:macro name="imu" params="name parent *joint_pose">

File: panther_description/urdf/panther.urdf.xacro (robot description, xacro)
@@ -30,6 +30,6 @@
   <xacro:include filename="$(find panther_description)/urdf/chassis.urdf.xacro" />
   <xacro:include filename="$(find panther_description)/urdf/track.urdf.xacro" />
-  <!--<xacro:include filename="$(find panther_description)/urdf/zedcamera.urdf.xacro" />
-  <xacro:include filename="$(find panther_description)/urdf/imu.urdf.xacro" />-->
+  <xacro:include filename="$(find panther_description)/urdf/zedcamera.urdf.xacro" />
+  <xacro:include filename="$(find panther_description)/urdf/imu.urdf.xacro" />
   <!-- Included URDF/XACRO Files -->
   <!-- Global properties -->
@@ -56,5 +56,5 @@
                                izz="1" />
     </inertial>
-    <!--<visual>
+    <visual>
       <origin xyz="0 0 0" rpy="0 0 0" />
       <geometry>
@@ -62,5 +62,5 @@
       </geometry>
       <material name="Green" />
-    </visual>-->
+    </visual>
   </link>
   <!-- Chassis -->
@@ -70,12 +70,12 @@
   <!-- Chassis - END -->
   <!-- ZED -->
-  <!--<xacro:zedcamera parent="frame_link">
-    <origin xyz="0.03600 0 0.1900" rpy="0 0 -1.5707963267949" />
-  </xacro:zedcamera>-->
+  <xacro:zedcamera parent="frame_link">
+    <origin xyz="-0.03600 0 0.1900" rpy="${M_PI} ${M_PI} ${-M_PI/2}" />
+  </xacro:zedcamera>
   <!-- ZED - END -->
   <!-- IMU -->
-  <!--<xacro:imu name="base_imu" parent="frame_link">
-    <origin xyz="0.0420817256507905 0 0.091441320597534" rpy="${M_PI} ${M_PI/2} 0" />
-  </xacro:imu>-->
+  <xacro:imu name="base_imu" parent="frame_link">
+    <origin xyz="-0.0420817256507905 0 0.091441320597534" rpy="0 ${M_PI/2} 0" />
+  </xacro:imu>
   <!-- IMU -->
   <!-- Track -->

File: panther_description/urdf/track.urdf.xacro (robot description, xacro)
@@ -197,5 +197,5 @@
   <xacro:gear type="${type}" orientation="${orientation}" />
   <!-- Passive wheels -->
-  <xacro:wheel type="${type}" orientation="${orientation}" conf="front_down" name="wheel_front_link" passive_wheel_type="continuous">
+  <xacro:wheel type="${type}" orientation="${orientation}" conf="front_down" name="wheel_front_link" wheel_radius="0.025" passive_wheel_type="continuous">
       <!-- visual wheel origin offest-->
       <origin xyz="0 0 0.020143" rpy="0 0 0" />
@@ -207,5 +207,5 @@
       <cylinder length="0.05" radius="0.025"/>
   </xacro:wheel>
-  <xacro:wheel type="${type}" orientation="${orientation}" conf="front_up" name="wheel_front_link" passive_wheel_type="continuous">
+  <xacro:wheel type="${type}" orientation="${orientation}" conf="front_up" name="wheel_front_link" wheel_radius="0.025" passive_wheel_type="continuous">
       <!-- visual wheel origin offest-->
       <origin xyz="0 0 0.020143" rpy="0 0 0" />
@@ -217,5 +217,5 @@
       <cylinder length="0.05" radius="0.025"/>
   </xacro:wheel>
-  <xacro:wheel type="${type}" orientation="${orientation}" conf="center_up" name="wheel_center_up_link" passive_wheel_type="continuous">
+  <xacro:wheel type="${type}" orientation="${orientation}" conf="center_up" name="wheel_center_up_link" wheel_radius="0.016" passive_wheel_type="continuous">
       <!-- visual wheel origin offest-->
       <origin xyz="0 0 0" rpy="0 0 0" />
@@ -227,5 +227,5 @@
       <cylinder length="0.05" radius="0.016"/>
   </xacro:wheel>
-  <xacro:wheel type="${type}" orientation="${orientation}" conf="center_A" name="wheel_center_link" passive_wheel_type="continuous">
+  <xacro:wheel type="${type}" orientation="${orientation}" conf="center_A" name="wheel_center_link" wheel_radius="0.016" passive_wheel_type="continuous">
       <!-- visual wheel origin offest-->
       <origin xyz="0 0 0" rpy="0 0 0" />
@@ -237,5 +237,5 @@
       <cylinder length="0.01" radius="0.016"/>
   </xacro:wheel>
-  <xacro:wheel type="${type}" orientation="${orientation}" conf="center_B" name="wheel_center_link" passive_wheel_type="continuous">
+  <xacro:wheel type="${type}" orientation="${orientation}" conf="center_B" name="wheel_center_link" wheel_radius="0.016" passive_wheel_type="continuous">
       <!-- visual wheel origin offest-->
       <origin xyz="0 0 0" rpy="0 0 0" />
@@ -247,5 +247,5 @@
       <cylinder length="0.01" radius="0.016"/>
   </xacro:wheel>
-  <xacro:wheel type="${type}" orientation="${orientation}" conf="center_C" name="wheel_center_link" passive_wheel_type="continuous">
+  <xacro:wheel type="${type}" orientation="${orientation}" conf="center_C" name="wheel_center_link" wheel_radius="0.016" passive_wheel_type="continuous">
       <!-- visual wheel origin offest-->
       <origin xyz="0 0 0" rpy="0 0 0" />
@@ -257,5 +257,5 @@
       <cylinder length="0.01" radius="0.016"/>
   </xacro:wheel>
-  <xacro:wheel type="${type}" orientation="${orientation}" conf="center_D" name="wheel_center_link" passive_wheel_type="continuous">
+  <xacro:wheel type="${type}" orientation="${orientation}" conf="center_D" name="wheel_center_link" wheel_radius="0.016" passive_wheel_type="continuous">
       <!-- visual wheel origin offest-->
       <origin xyz="0 0 0" rpy="0 0 0" />

File: panther_description/urdf/wheel.urdf.xacro (robot description, xacro)
@@ -26,5 +26,5 @@
 -->
 <robot xmlns:xacro="http://ros.org/wiki/xacro" name="wheel">
-  <xacro:macro name="wheel" params="type orientation conf name passive_wheel_type *visual_pose *wheel_pose *collision_shape">
+  <xacro:macro name="wheel" params="type orientation conf name passive_wheel_type wheel_radius *visual_pose *wheel_pose *collision_shape">
   <!-- Front passive wheel all time type continous -->
   <link name="wheel_${type}_${conf}_Link">
@@ -57,5 +57,5 @@
     <!-- Passive sprocket rotate automatically according to the status of the active one -->
     <xacro:if value="${passive_wheel_type == 'continuous'}">
-      <mimic joint="${type}_joint" multiplier="1" offset="0"/>
+      <mimic joint="${type}_joint" multiplier="${sprocket_radius/wheel_radius}" offset="0"/>
     </xacro:if>
   </joint>

File: panther_description/urdf/zedcamera.urdf.xacro (robot description, xacro)
@@ -1,3 +1,28 @@
 <?xml version="1.0"?>
+<!--
+Copyright (C) 2017, Raffaello Bonghi <raffaello@rnext.it>
+All rights reserved
+Redistribution and use in source and binary forms, with or without
+modification, are permitted provided that the following conditions are met:
+1. Redistributions of source code must retain the above copyright
+   notice, this list of conditions and the following disclaimer.
+2. Redistributions in binary form must reproduce the above copyright
+   notice, this list of conditions and the following disclaimer in the
+   documentation and/or other materials provided with the distribution.
+3. Neither the name of the copyright holder nor the names of its
+   contributors may be used to endorse or promote products derived
+   from this software without specific prior written permission.
+THIS SOFTWARE IS PROVIDED BY THE COPYRIGHT HOLDERS AND
+CONTRIBUTORS "AS IS" AND ANY EXPRESS OR IMPLIED WARRANTIES, INCLUDING,
+BUT NOT LIMITED TO, THE IMPLIED WARRANTIES OF MERCHANTABILITY AND FITNESS
+FOR A PARTICULAR PURPOSE ARE DISCLAIMED. IN NO EVENT SHALL THE COPYRIGHT
+HOLDER OR CONTRIBUTORS BE LIABLE FOR ANY DIRECT, INDIRECT, INCIDENTAL,
+SPECIAL, EXEMPLARY, OR CONSEQUENTIAL DAMAGES (INCLUDING, BUT NOT LIMITED TO,
+PROCUREMENT OF SUBSTITUTE GOODS OR SERVICES; LOSS OF USE, DATA, OR PROFITS;
+OR BUSINESS INTERRUPTION) HOWEVER CAUSED AND ON ANY THEORY OF LIABILITY,
+WHETHER IN CONTRACT, STRICT LIABILITY, OR TORT (INCLUDING NEGLIGENCE
+OR OTHERWISE) ARISING IN ANY WAY OUT OF THE USE OF THIS SOFTWARE,
+EVEN IF ADVISED OF THE POSSIBILITY OF SUCH DAMAGE.
+-->
 <robot name="zedcamera" xmlns:xacro="http://ros.org/wiki/xacro">
 <xacro:property name="optical_y_offset" value="0.06" />

Commit message: Improve and fix panther_description

File: panther_description/urdf/chassis.urdf.xacro (robot description, xacro)
@@ -1,5 +1,5 @@
 <?xml version="1.0"?>
 <!--
-Copyright (C) 2017, Raffaello Bonghi <raffaello@rnext.it>
+Copyright (C) 2020, Raffaello Bonghi <raffaello@rnext.it>
 All rights reserved
 Redistribution and use in source and binary forms, with or without
@@ -29,9 +29,9 @@
   <link name="frame_link">
     <inertial>
-      <origin xyz="0.00103 0.0004 0.058" rpy="0 0 0" />
-      <mass value="1.147" />
-      <inertia ixx="0.011143732226453" ixy="2.27736840022485E-05" ixz="0.000768863495805356"
-        iyy="0.0184528503285751" iyz="2.40527095667182E-05"
-        izz="0.0219088128480578" />
+      <origin xyz="0 0 0" rpy="0 0 0" />
+      <mass value="11.0" />
+      <inertia ixx="1" ixy="0" ixz="0"
+                       iyy="1" iyz="0"
+                               izz="1" />
     </inertial>
     <visual>

File: panther_description/urdf/panther.urdf.xacro (robot description, xacro)
@@ -1,5 +1,5 @@
 <?xml version="1.0"?>
 <!--
-Copyright (C) 2017, Raffaello Bonghi <raffaello@rnext.it>
+Copyright (C) 2020, Raffaello Bonghi <raffaello@rnext.it>
 All rights reserved
 Redistribution and use in source and binary forms, with or without
@@ -25,5 +25,5 @@
 EVEN IF ADVISED OF THE POSSIBILITY OF SUCH DAMAGE.
 -->
-<robot name="panther_robot" xmlns:xacro="http://ros.org/wiki/xacro">
+<robot name="panther" xmlns:xacro="http://ros.org/wiki/xacro">
   <!-- Included URDF/XACRO Files -->
   <xacro:include filename="$(find panther_description)/urdf/materials.urdf" />
@@ -46,14 +46,6 @@
   <xacro:property name="wheel_offset_z" value="${wheel_radius}"/>
   <!-- Sprocket and gear properties -->
-  <xacro:macro name="panther_robot">
   <!-- base_link -->
   <link name="base_link">
-    <inertial>
-      <origin xyz="0 0 0" rpy="0 0 0" />
-      <mass value="11.0" />
-      <inertia ixx="1" ixy="0" ixz="0"
-                       iyy="1" iyz="0"
-                               izz="1" />
-    </inertial>
     <visual>
       <origin xyz="0 0 0" rpy="0 0 0" />
@@ -83,4 +75,3 @@
   <xacro:track type="right" parent="frame_link" />
   <!-- Track - END -->
-  </xacro:macro>
 </robot>
