Commit message: Improved panther xacro

File: panther_description/urdf/panther.urdf.xacro (robot description, xacro)
@@ -3,4 +3,5 @@
   <!-- Included URDF/XACRO Files -->
   <xacro:include filename="$(find panther_description)/urdf/materials.urdf" />
+  <xacro:include filename="$(find panther_description)/urdf/track.urdf.xacro" />
   <!-- Included URDF/XACRO Files -->
   <!-- Global properties -->
@@ -8,375 +9,17 @@
   <property name="M_PI" value="3.14159"/>
   <!-- Global properties -->
- <xacro:macro name="panther_robot">
+  <xacro:macro name="panther_robot">
   <!-- base_link -->
   <link name="base_link">
   </link>
-  <link name="track_link">
-    <inertial>
-      <origin xyz="-0.0168 0.0080 0.0061" rpy="0 0 0" />
-      <mass value="0.512" />
-      <inertia ixx="0.0008" ixy="0" ixz="0"
-        iyy="0.005" iyz="0.0001"
-        izz="0.005" />
-    </inertial>
-    <visual>
-      <origin xyz="0 0 0" rpy="0 0 0" />
-      <geometry>
-        <mesh filename="${path_meshes}/track/left/track_link.STL" />
-      </geometry>
-      <material name="White-Alpha" />
-    </visual>
-  </link>
-  <joint name="track_joint" type="fixed">
-    <origin xyz="0 0 0" rpy="0 0 0" />
-    <parent link="base_link" />
-    <child link="track_link" />
-    <axis xyz="0 0 0" />
-  </joint>
-  <link name="iron_Link">
-    <inertial>
-      <origin xyz="0.028 0.026 0.011" rpy="0 0 0" />
-      <mass value="1.412" />
-      <inertia ixx="0.0021" ixy="0.0009" ixz="0.0003"
-        iyy="0.0080" iyz="0.0002"
-        izz="0.009" />
-    </inertial>
-    <visual>
-      <origin xyz="0 0 0" rpy="0 0 0" />
-      <geometry>
-        <mesh filename="${path_meshes}/track/left/iron_link.STL" />
-      </geometry>
-      <material name="GunMetalGrey" />
-    </visual>
-  </link>
-  <joint name="iron_joint" type="fixed">
-    <origin xyz="0 0 0" rpy="0 0 0" />
-    <parent link="track_link" />
-    <child link="iron_Link" />
-    <axis xyz="0 0 0" />
-  </joint>
-  <link name="damper_Link">
-    <inertial>
-      <origin xyz="0.011 0.014 0.028" rpy="0 0 0" />
-      <mass value="0.028" />
-      <inertia ixx="0" ixy="0" ixz="0"
-        iyy="0.0007" iyz="0"
-        izz="0.0002" />
-    </inertial>
-    <visual>
-      <origin xyz="0 0 0" rpy="0 0 0" />
-      <geometry>
-        <mesh filename="${path_meshes}/track/left/damper_link.STL" />
-      </geometry>
-      <material name="Black" />
-    </visual>
-  </link>
-  <joint name="damper_joint" type="fixed">
-    <origin xyz="0 0 0" rpy="0 0 0" />
-    <parent link="track_link" />
-    <child link="damper_Link" />
-    <axis xyz="0 0 0" />
-  </joint>
-  <link name="damper_label_Link">
-    <inertial>
-      <origin xyz="0.0111 0.0137 0.0341" rpy="0 0 0" />
-      <mass value="0.0062" />
-      <inertia ixx="0" ixy="0" ixz="0"
-        iyy="0" iyz="0"
-        izz="0" />
-    </inertial>
-    <visual>
-      <origin xyz="0 0 0" rpy="0 0 0" />
-      <geometry>
-        <mesh filename="${path_meshes}/track/left/damper_label_link.STL" />
-      </geometry>
-      <material name="Green" />
-    </visual>
-  </link>
-  <joint name="damper_label_joint" type="fixed">
-    <origin xyz="0 0 0" rpy="0 0 0" />
-    <parent link="damper_Link" />
-    <child link="damper_label_Link" />
-    <axis xyz="0 0 0" />
-  </joint>
-  <link name="fender_Link">
-    <inertial>
-      <origin xyz="-0.0044 0.0167 0.0872" rpy="0 0 0" />
-      <mass value="0.0853" />
-      <inertia ixx="0" ixy="0" ixz="0"
-        iyy="0.0007" iyz="0"
-        izz="0.0007" />
-    </inertial>
-    <visual>
-      <origin xyz="0 0 0" rpy="0 0 0" />
-      <geometry>
-        <mesh filename="${path_meshes}/track/left/fender_link.STL" />
-      </geometry>
-      <material name="Black" />
-    </visual>
-  </link>
-  <joint name="fender_joint" type="fixed">
-    <origin xyz="0 0 0" rpy="0 0 0" />
-    <parent link="track_link" />
-    <child link="fender_Link" />
-    <axis xyz="0 0 0" />
-  </joint>
-  <link name="rubber_Link">
-    <inertial>
-      <origin xyz="-0.0137 0 -0.0014" rpy="0 0 0" />
-      <mass value="0.466" />
-      <inertia ixx="0.0016" ixy="0" ixz="-0.0003"
-        iyy="0.0090" iyz="0"
-        izz="0.007" />
-    </inertial>
-    <visual>
-      <origin xyz="0 0 0" rpy="0 0 0" />
-      <geometry>
-        <mesh filename="${path_meshes}/track/left/rubber_link.STL" />
-      </geometry>
-      <material name="Black" />
-    </visual>
-  </link>
-  <joint name="rubber_joint" type="fixed">
-    <origin xyz="0 0 0" rpy="0 0 0" />
-    <parent link="track_link" />
-    <child link="rubber_Link" />
-    <axis xyz="0 0 0" />
-  </joint>
-  <link name="chain_Link">
-    <inertial>
-      <origin xyz="0.101 0.0001 -0.0026" rpy="0 0 0" />
-      <mass value="0.0708" />
-      <inertia ixx="0" ixy="0" ixz="0"
-        iyy="0" iyz="0"
-        izz="0.0001" />
-    </inertial>
-    <visual>
-      <origin xyz="0 0 0" rpy="0 0 0" />
-      <geometry>
-        <mesh filename="${path_meshes}/track/left/chain_link.STL" />
-      </geometry>
-      <material name="DarkGrey" />
-    </visual>
-  </link>
-  <joint name="chain_joint" type="fixed">
-    <origin xyz="0 0 0" rpy="0 0 0" />
-    <parent link="track_link" />
-    <child link="chain_Link" />
-    <axis xyz="0 0 0" />
-  </joint>
-  <!-- PASSIVE WHEELS -->
-  <link name="wheel_center_up_Link">
-    <inertial>
-      <origin xyz="0 0 0" rpy="0 0 0" />
-      <mass value="0.016" />
-      <inertia ixx="0" ixy="0" ixz="0"
-        iyy="0" iyz="0"
-        izz="0" />
-    </inertial>
-    <visual>
-      <origin xyz="0 0 0" rpy="0 0 0" />
-      <geometry>
-        <mesh filename="${path_meshes}/track/wheel_center_up_link.STL" />
-      </geometry>
-      <material name="White-Alpha" />
-    </visual>
-  </link>
-  <joint name="wheel_center_up_joint" type="continuous">
-    <origin
-      xyz="0 0 0.0735790044064745"
-      rpy="1.5707963267949 -0.800774112020821 6.31428234397228E-17" />
-    <parent link="track_link" />
-    <child link="wheel_center_up_Link" />
-    <axis xyz="0 0 -1" />
-  </joint>
-  <link name="wheel_front_up_Link">
-    <inertial>
-      <origin xyz="0 0 -0.020143" rpy="0 0 0" />
-      <mass value="0.043" />
-      <inertia ixx="0" ixy="0" ixz="0"
-        iyy="0" iyz="0"
-        izz="0" />
-    </inertial>
-    <visual>
-      <origin xyz="0 0 0" rpy="0 0 0" />
-      <geometry>
-        <mesh filename="${path_meshes}/track/wheel_front_link.STL" />
-      </geometry>
-      <material name="White-Alpha" />
-    </visual>
-  </link>
-  <joint name="wheel_front_up_joint" type="continuous">
-    <origin
-      xyz="-0.18867 -0.020143 0.010536"
-      rpy="-1.5708 -0.13483 3.1416" />
-    <parent link="track_link" />
-    <child link="wheel_front_up_Link" />
-    <axis xyz="0 0 -1" />
-  </joint>
-  <link name="wheel_front_down_Link">
-    <inertial>
-      <origin xyz="0 0 -0.020143" rpy="0 0 0" />
-      <mass value="0.0431" />
-      <inertia ixx="0" ixy="0" ixz="0"
-        iyy="0" iyz="0"
-        izz="0" />
-    </inertial>
-    <visual>
-      <origin xyz="0 0 0" rpy="0 0 0" />
-      <geometry>
-        <mesh filename="${path_meshes}/track/wheel_front_link.STL" />
-      </geometry>
-      <material name="White-Alpha" />
-    </visual>
-  </link>
-  <joint name="wheel_front_down_joint" type="continuous">
-    <origin
-      xyz="-0.15659 -0.020143 -0.034143"
-      rpy="1.5708 -0.36637 2.3494E-17" />
-    <parent link="track_link" />
-    <child link="wheel_front_down_Link" />
-    <axis xyz="0 0 -1" />
-  </joint>
-  <link name="wheel_center_A_Link">
-    <inertial>
-      <origin xyz="-0.064 -0.046 0.004" rpy="0 0 0" />
-      <mass value="0.0082" />
-      <inertia ixx="0" ixy="0" ixz="0"
-        iyy="0" iyz="0"
-        izz="0" />
-    </inertial>
-    <visual>
-      <origin xyz="0 0 0" rpy="0 0 0" />
-      <geometry>
-        <mesh filename="${path_meshes}/track/wheel_center_link.STL" />
-      </geometry>
-      <material name="White-Alpha" />
-    </visual>
-  </link>
-  <joint name="wheel_center_A_joint" type="continuous">
-    <!-- <origin xyz="-0.065 0.004 0.005" rpy="1.5708 0 0" />-->
-    <origin xyz="-0.065 -0.004 -0.042" rpy="1.5708 0 0" />
-    <parent link="track_link" />
-    <child link="wheel_center_A_Link" />.
-    <axis xyz="0 0 -1" />
-  </joint>
-  <link name="wheel_center_B_Link">
-    <inertial>
-      <origin xyz="-0.020 -0.0465 0.004" rpy="0 0 0" />
-      <mass value="0.0083" />
-      <inertia ixx="0" ixy="0" ixz="0"
-        iyy="0" iyz="0"
-        izz="0" />
-    </inertial>
-    <visual>
-      <origin xyz="0 0 0" rpy="0 0 0" />
-      <geometry>
-        <mesh filename="${path_meshes}/track/wheel_center_link.STL" />
-      </geometry>
-      <material name="White-Alpha" />
-    </visual>
-  </link>
-  <joint name="wheel_center_B_joint" type="continuous">
-    <origin xyz="-0.020 -0.004 -0.042" rpy="1.5708 0 0" />
-    <parent link="track_link" />
-    <child link="wheel_center_B_Link" />
-    <axis xyz="0 0 -1" />
-  </joint>
-  <link name="wheel_center_C_Link">
-    <inertial>
-      <origin xyz="0.020 -0.0462 0.004" rpy="0 0 0" />
-      <mass value="0.0083" />
-      <inertia ixx="0" ixy="0" ixz="0"
-        iyy="0" iyz="0"
-        izz="0" />
-    </inertial>
-    <visual>
-      <origin
-        xyz="0 0 0"
-        rpy="0 0 0" />
-      <geometry>
-        <mesh filename="${path_meshes}/track/wheel_center_link.STL" />
-      </geometry>
-      <material name="White-Alpha" />
-    </visual>
-  </link>
-  <joint name="wheel_center_C_joint" type="continuous">
-    <origin xyz="0.020 -0.004 -0.042" rpy="1.5708 0 0" />
-    <parent link="track_link" />
-    <child link="wheel_center_C_Link" />
-    <axis xyz="0 0 -1" />
-  </joint>
-  <link name="wheel_center_D_Link">
-    <inertial>
-      <origin xyz="0.0648 -0.0462 0.004" rpy="0 0 0" />
-      <mass value="0.0083" />
-      <inertia ixx="0" ixy="0" ixz="0"
-        iyy="0" iyz="0"
-        izz="0" />
-    </inertial>
-    <visual>
-      <origin xyz="0 0 0" rpy="0 0 0" />
-      <geometry>
-        <mesh filename="${path_meshes}/track/wheel_center_link.STL" />
-      </geometry>
-      <material name="White-Alpha" />
-    </visual>
-  </link>
-  <joint name="wheel_center_D_joint" type="continuous">
-    <origin xyz="0.065 -0.004 -0.042" rpy="1.5707963267949 0 0" />
-    <parent link="track_link" />
-    <child link="wheel_center_D_Link" />
-    <axis xyz="0 0 -1" />
-  </joint>
-  <!-- TRACTION WHEELS -->
-  <link name="gear_Link">
-    <inertial>
-      <origin xyz="0 0 0.008" rpy="0 0 0" />
-      <mass value="0.0111" />
-      <inertia ixx="0" ixy="0" ixz="0"
-        iyy="0" iyz="0"
-        izz="0" />
-    </inertial>
-    <visual>
-      <origin xyz="0 0 0" rpy="0 0 0" />
-      <geometry>
-        <mesh filename="${path_meshes}/track/gear_link.STL" />
-      </geometry>
-      <material name="DarkGrey" />
-    </visual>
-  </link>
-  <joint name="gear_joint" type="continuous">
-    <origin
-      xyz="0.0536535102814494 -0.00979339452125411 0.0186240655062149"
-      rpy="-1.5707963267949 -1.50760970347625 3.14159265358979" />
-    <parent link="track_link" />
-    <child link="gear_Link" />
-    <axis xyz="0 0 -1" />
-  </joint>
-  <link name="sprocket_Link">
-    <inertial>
-      <origin xyz="0 0 -0.0167" rpy="0 0 0" />
-      <mass value="0.098" />
-      <inertia ixx="0" ixy="0" ixz="0"
-        iyy="0" iyz="0"
-        izz="0" />
-    </inertial>
-    <visual>
-      <origin xyz="0 0 0" rpy="0 0 0" />
-      <geometry>
-        <mesh filename="${path_meshes}/track/sprocket_link.STL" />
-      </geometry>
-      <material name="Black" />
-    </visual>
-  </link>
-  <joint name="sprocket_joint" type="continuous">
-    <origin
-      xyz="0.15476 -0.020382 -0.026643"
-      rpy="1.5708 -1.5708 0" />
-    <parent link="track_link" />
-    <child link="sprocket_Link" />
-    <axis xyz="0 0 -1" />
-  </joint>
+  <!-- Track -->
+   <!-- passive_wheel_type tye: (1) continuous or (2) fixed -->
+  <xacro:track position="left" parent="base_link" passive_wheel_type="fixed">
+    <origin xyz="0 -0.2 0" rpy="0 0 0" />
+  </xacro:track>
+  <xacro:track position="right" parent="base_link" passive_wheel_type="fixed">
+    <origin xyz="0 0.2 0" rpy="0 0 0" />
+  </xacro:track>
+  <!-- Track - END -->
   </xacro:macro>
 </robot>

Commit message: Added chassis Panther

File: panther_description/urdf/panther.urdf.xacro (robot description, xacro)
@@ -4,4 +4,6 @@
   <xacro:include filename="$(find panther_description)/urdf/materials.urdf" />
   <xacro:include filename="$(find panther_description)/urdf/track.urdf.xacro" />
+  <xacro:include filename="$(find panther_description)/urdf/chassis.urdf.xacro" />
+  <xacro:include filename="$(find panther_description)/urdf/zedcamera.urdf.xacro" />
   <!-- Included URDF/XACRO Files -->
   <!-- Global properties -->
@@ -12,12 +14,29 @@
   <!-- base_link -->
   <link name="base_link">
+    <visual>
+      <origin xyz="0 0 0" rpy="0 0 0" />
+      <geometry>
+        <cylinder length="0.001" radius="0.05"/>
+      </geometry>
+      <material name="Green" />
+    </visual>
   </link>
+  <!-- Chassis -->
+  <xacro:chassis parent="base_link">
+    <origin xyz="0 0 0.08" rpy="0 0 3.14159" />
+  </xacro:chassis>
+  <!-- Chassis - END -->
+  <!-- ZED -->
+  <xacro:zedcamera parent="frame_link">
+    <origin xyz="0.03600 0 0.1900" rpy="0 0 -1.5707963267949" />
+  </xacro:zedcamera>
+  <!-- ZED - END -->
   <!-- Track -->
-   <!-- passive_wheel_type tye: (1) continuous or (2) fixed -->
-  <xacro:track position="left" parent="base_link" passive_wheel_type="fixed">
-    <origin xyz="0 -0.2 0" rpy="0 0 0" />
+  <!-- passive_wheel_type tye: (1) continuous or (2) fixed -->
+  <xacro:track position="left" parent="frame_link" passive_wheel_type="fixed">
+    <origin xyz="0 -0.161 -0.014" rpy="0 0 0" />
   </xacro:track>
-  <xacro:track position="right" parent="base_link" passive_wheel_type="fixed">
-    <origin xyz="0 0.2 0" rpy="0 0 0" />
+  <xacro:track position="right" parent="frame_link" passive_wheel_type="fixed">
+    <origin xyz="0 0.161 -0.014" rpy="0 0 0" />
   </xacro:track>
   <!-- Track - END -->

File: panther_description/urdf/track.urdf.xacro (robot description, xacro)
@@ -83,5 +83,5 @@
         <mesh filename="${path_meshes}/track/${position}/damper_label_link.STL" />
       </geometry>
-      <material name="Green" />
+      <material name="Pink" />
     </visual>
   </link>

Commit message: Fixed deprecated syntax xacro

File: panther_description/urdf/panther.urdf.xacro (robot description, xacro)
@@ -8,6 +8,6 @@
   <!-- Included URDF/XACRO Files -->
   <!-- Global properties -->
-  <property name="path_meshes" value="package://panther_description/meshes"/>
-  <property name="M_PI" value="3.14159"/>
+  <xacro:property name="path_meshes" value="package://panther_description/meshes"/>
+  <xacro:property name="M_PI" value="3.14159"/>
   <!-- Global properties -->
   <xacro:macro name="panther_robot">

Commit message: Fixed information referece sprocket and added rviz image

File: panther_description/urdf/panther.urdf.xacro (robot description, xacro)
@@ -5,4 +5,6 @@
   <xacro:include filename="$(find panther_description)/urdf/track.urdf.xacro" />
   <xacro:include filename="$(find panther_description)/urdf/chassis.urdf.xacro" />
+  <xacro:include filename="$(find panther_description)/urdf/sprocket.urdf.xacro" />
+  <xacro:include filename="$(find panther_description)/urdf/gear.urdf.xacro" />
   <xacro:include filename="$(find panther_description)/urdf/zedcamera.urdf.xacro" />
   <!-- Included URDF/XACRO Files -->
@@ -11,4 +13,13 @@
   <xacro:property name="M_PI" value="3.14159"/>
   <!-- Global properties -->
+  <!-- Sprocket and gear properties -->
+  <xacro:property name="sprocket_radius" value="0.0325"/>
+  <xacro:property name="sprocket_leght" value="0.05"/>
+  <xacro:property name="sprocket_teeth" value="24"/>
+  <xacro:property name="gear_teeth" value="16"/>
+  <xacro:property name="wheel_offset_x" value="-0.00"/>
+  <xacro:property name="wheel_offset_y" value="0.08"/>
+  <xacro:property name="wheel_offset_z" value="${wheel_radius}"/>
+  <!-- Sprocket and gear properties -->
   <xacro:macro name="panther_robot">
   <!-- base_link -->
@@ -41,4 +52,20 @@
   </xacro:track>
   <!-- Track - END -->
+  <!-- Sprocket -->
+  <xacro:sprocket name="Left" position="left" parent="track_left_link">
+    <origin xyz="0 -0.161 -0.014" rpy="0 0 0" />
+  </xacro:sprocket>
+  <xacro:sprocket name="Right" position="right" parent="track_right_link">
+    <origin xyz="0 0.161 -0.014" rpy="0 0 0" />
+  </xacro:sprocket>
+  <!-- Sprocket - END -->
+  <!-- Gear -->
+  <xacro:gear name="Left" position="left" parent="track_left_link">
+    <origin xyz="0 -0.161 -0.014" rpy="0 0 0" />
+  </xacro:gear>
+  <xacro:gear name="Right" position="right" parent="track_right_link">
+    <origin xyz="0 0.161 -0.014" rpy="0 0 0" />
+  </xacro:gear>
+  <!-- Gear - END -->
   </xacro:macro>
 </robot>

File: panther_description/urdf/track.urdf.xacro (robot description, xacro)
@@ -322,5 +322,5 @@
   </joint>
   <!-- TRACTION WHEELS -->
-  <link name="gear_${position}_Link">
+<!--  <link name="gear_${position}_Link">
     <inertial>
       <origin xyz="0 0 0.008" rpy="0 0 0" />
@@ -352,6 +352,6 @@
     <child link="gear_${position}_Link" />
     <axis xyz="0 0 -1" />
-  </joint>
-  <link name="sprocket_${position}_Link">
+  </joint>-->
+<!--  <link name="sprocket_${position}_Link">
     <inertial>
       <origin xyz="0 0 -0.0167" rpy="0 0 0" />
@@ -383,5 +383,5 @@
     <child link="sprocket_${position}_Link" />
     <axis xyz="0 0 -1" />
-  </joint>
+  </joint>-->
   </xacro:macro>
 </robot>

Commit message: Fixed IMU

File: panther_description/urdf/panther.urdf.xacro (robot description, xacro)
@@ -46,5 +46,6 @@
   <!-- IMU -->
   <xacro:imu name="base_imu" parent="frame_link">
-    <origin xyz="0.0420817256507905 0 0.091441320597534" rpy="${M_PI} ${M_PI/2} 0" />
+    <!--<origin xyz="0.0420817256507905 0 0.091441320597534" rpy="${M_PI} ${M_PI/2} 0" />-->
+    <origin xyz="0.0420817256507905 0 0.091441320597534" rpy="${-M_PI/2} 0 ${M_PI/2}" />
   </xacro:imu>
   <!-- IMU -->
