Commit message: Added gazebo reference

File: panther_description/urdf/panther.urdf.xacro (robot description, xacro)
@@ -46,32 +46,32 @@
   <!-- IMU -->
   <xacro:imu name="base_imu" parent="frame_link">
-    <!--<origin xyz="0.0420817256507905 0 0.091441320597534" rpy="${M_PI} ${M_PI/2} 0" />-->
-    <origin xyz="0.0420817256507905 0 0.091441320597534" rpy="${-M_PI/2} 0 ${M_PI/2}" />
+    <origin xyz="0.0420817256507905 0 0.091441320597534" rpy="${M_PI} ${M_PI/2} 0" />
+    <!--<origin xyz="0.0420817256507905 0 0.091441320597534" rpy="${-M_PI/2} 0 ${M_PI/2}" />-->
   </xacro:imu>
   <!-- IMU -->
   <!-- Track -->
-  <!-- passive_wheel_type tye: (1) continuous or (2) fixed -->
-  <xacro:track position="left" parent="frame_link" passive_wheel_type="fixed">
+  <!-- passive_wheel_type type: (1) continuous or (2) fixed -->
+  <xacro:track name="Left" position="left" parent="frame_link" passive_wheel_type="fixed">
     <origin xyz="0 -0.161 -0.014" rpy="0 0 0" />
   </xacro:track>
-  <xacro:track position="right" parent="frame_link" passive_wheel_type="fixed">
+  <xacro:track name="Right" position="right" parent="frame_link" passive_wheel_type="fixed">
     <origin xyz="0 0.161 -0.014" rpy="0 0 0" />
   </xacro:track>
   <!-- Track - END -->
   <!-- Sprocket -->
-  <xacro:sprocket name="Left" position="left" parent="track_left_link">
+  <!--<xacro:sprocket name="Left" position="left" parent="track_left_link">
     <origin xyz="0 -0.161 -0.014" rpy="0 0 0" />
   </xacro:sprocket>
   <xacro:sprocket name="Right" position="right" parent="track_right_link">
     <origin xyz="0 0.161 -0.014" rpy="0 0 0" />
-  </xacro:sprocket>
+  </xacro:sprocket>-->
   <!-- Sprocket - END -->
   <!-- Gear -->
-  <xacro:gear name="Left" position="left" parent="track_left_link">
+  <!--<xacro:gear name="Left" position="left" parent="track_left_link">
     <origin xyz="0 -0.161 -0.014" rpy="0 0 0" />
   </xacro:gear>
   <xacro:gear name="Right" position="right" parent="track_right_link">
     <origin xyz="0 0.161 -0.014" rpy="0 0 0" />
-  </xacro:gear>
+  </xacro:gear>-->
   <!-- Gear - END -->
   </xacro:macro>

File: panther_description/urdf/track.urdf.xacro (robot description, xacro)
@@ -2,5 +2,5 @@
 <robot xmlns:xacro="http://ros.org/wiki/xacro" name="track">
  <!-- passive_wheel_type tye: (1) continuous or (2) fixed -->
- <xacro:macro name="track" params="position parent passive_wheel_type *joint_pose">
+ <xacro:macro name="track" params="name position parent passive_wheel_type *joint_pose">
   <!-- TRACK FIXED LINKS -->
   <link name="track_${position}_link">
@@ -207,4 +207,5 @@
     <axis xyz="0 0 -1" />
   </joint>
+  <!-- Front passive wheel all time type continous -->
   <link name="wheel_${position}_front_down_Link">
     <inertial>
@@ -222,6 +223,12 @@
       <material name="White-Alpha" />
     </visual>
-  </link>
-  <joint name="wheel_${position}_front_down_joint" type="${passive_wheel_type}">
+    <collision>
+      <origin xyz="0 0 -0.025" rpy="0 0 0" />
+      <geometry>
+        <cylinder length="0.05" radius="0.025"/>
+      </geometry>
+    </collision>
+  </link>
+  <joint name="wheel_${position}_front_down_joint" type="continuous">
     <origin
       xyz="-0.15659 -0.020143 -0.034143"
@@ -321,67 +328,14 @@
     <axis xyz="0 0 -1" />
   </joint>
-  <!-- TRACTION WHEELS -->
-<!--  <link name="gear_${position}_Link">
-    <inertial>
-      <origin xyz="0 0 0.008" rpy="0 0 0" />
-      <mass value="0.0111" />
-      <inertia ixx="0" ixy="0" ixz="0"
-        iyy="0" iyz="0"
-        izz="0" />
-    </inertial>
-    <visual>
-      <origin xyz="0 0 0" rpy="0 0 0" />
-      <geometry>
-        <mesh filename="${path_meshes}/track/gear_link.STL" />
-      </geometry>
-      <material name="DarkGrey" />
-    </visual>
-  </link>
-  <joint name="gear_${position}_joint" type="continuous">
-    <xacro:if value="${position == 'left'}">
-    <origin
-      xyz="0.0536535102814494 -0.00979339452125411 0.0186240655062149"
-      rpy="-1.5707963267949 -1.50760970347625 3.14159265358979" />
-    </xacro:if>
-    <xacro:if value="${position == 'right'}">
-    <origin
-      xyz="0.0536535102814494 0.00979339452125411 0.0186240655062149"
-      rpy="1.5707963267949 -1.50760970347625 3.14159265358979" />
-    </xacro:if>
-    <parent link="track_${position}_link" />
-    <child link="gear_${position}_Link" />
-    <axis xyz="0 0 -1" />
-  </joint>-->
-<!--  <link name="sprocket_${position}_Link">
-    <inertial>
-      <origin xyz="0 0 -0.0167" rpy="0 0 0" />
-      <mass value="0.098" />
-      <inertia ixx="0" ixy="0" ixz="0"
-        iyy="0" iyz="0"
-        izz="0" />
-    </inertial>
-    <visual>
-      <origin xyz="0 0 0" rpy="0 0 0" />
-      <geometry>
-        <mesh filename="${path_meshes}/track/sprocket_link.STL" />
-      </geometry>
-      <material name="Black" />
-    </visual>
-  </link>
-  <joint name="sprocket_${position}_joint" type="continuous">
-    <xacro:if value="${position == 'left'}">
-    <origin
-      xyz="0.15476 -0.020382 -0.026643"
-      rpy="1.5708 -1.5708 0" />
-    </xacro:if>
-    <xacro:if value="${position == 'right'}">
-    <origin
-      xyz="0.15476 0.020382 -0.026643"
-      rpy="-1.5708 -1.5708 0" />
-    </xacro:if>
-    <parent link="track_${position}_link" />
-    <child link="sprocket_${position}_Link" />
-    <axis xyz="0 0 -1" />
-  </joint>-->
+  <!-- Sprocket -->
+  <xacro:sprocket name="${name}" position="${position}" parent="track_${position}_link">
+    <origin xyz="0 -0.161 -0.014" rpy="0 0 0" />
+  </xacro:sprocket>
+  <!-- Sprocket - END -->
+  <!-- Gear -->
+  <xacro:gear name="${name}" position="${position}" parent="track_${position}_link">
+    <origin xyz="0 -0.161 -0.014" rpy="0 0 0" />
+  </xacro:gear>
+  <!-- Gear - END -->
   </xacro:macro>
 </robot>

Commit message: Fixed panther gazebo description and added color

File: panther_description/urdf/panther.urdf.xacro (robot description, xacro)
@@ -1,3 +1,28 @@
 <?xml version="1.0"?>
+<!--
+Copyright (C) 2017, Raffaello Bonghi <raffaello@rnext.it>
+All rights reserved
+Redistribution and use in source and binary forms, with or without
+modification, are permitted provided that the following conditions are met:
+1. Redistributions of source code must retain the above copyright
+   notice, this list of conditions and the following disclaimer.
+2. Redistributions in binary form must reproduce the above copyright
+   notice, this list of conditions and the following disclaimer in the
+   documentation and/or other materials provided with the distribution.
+3. Neither the name of the copyright holder nor the names of its
+   contributors may be used to endorse or promote products derived
+   from this software without specific prior written permission.
+THIS SOFTWARE IS PROVIDED BY THE COPYRIGHT HOLDERS AND
+CONTRIBUTORS "AS IS" AND ANY EXPRESS OR IMPLIED WARRANTIES, INCLUDING,
+BUT NOT LIMITED TO, THE IMPLIED WARRANTIES OF MERCHANTABILITY AND FITNESS
+FOR A PARTICULAR PURPOSE ARE DISCLAIMED. IN NO EVENT SHALL THE COPYRIGHT
+HOLDER OR CONTRIBUTORS BE LIABLE FOR ANY DIRECT, INDIRECT, INCIDENTAL,
+SPECIAL, EXEMPLARY, OR CONSEQUENTIAL DAMAGES (INCLUDING, BUT NOT LIMITED TO,
+PROCUREMENT OF SUBSTITUTE GOODS OR SERVICES; LOSS OF USE, DATA, OR PROFITS;
+OR BUSINESS INTERRUPTION) HOWEVER CAUSED AND ON ANY THEORY OF LIABILITY,
+WHETHER IN CONTRACT, STRICT LIABILITY, OR TORT (INCLUDING NEGLIGENCE
+OR OTHERWISE) ARISING IN ANY WAY OUT OF THE USE OF THIS SOFTWARE,
+EVEN IF ADVISED OF THE POSSIBILITY OF SUCH DAMAGE.
+-->
 <robot name="panther_robot" xmlns:xacro="http://ros.org/wiki/xacro">
   <!-- Included URDF/XACRO Files -->
@@ -26,4 +51,11 @@
   <!-- base_link -->
   <link name="base_link">
+    <inertial>
+      <origin xyz="0 0 0" rpy="0 0 0" />
+      <mass value="11.0" />
+      <inertia ixx="1" ixy="0" ixz="0"
+                       iyy="1" iyz="0"
+                               izz="1" />
+    </inertial>
     <visual>
       <origin xyz="0 0 0" rpy="0 0 0" />
@@ -57,6 +89,9 @@
       rpy="0 0 0" />
     <origin
+      xyz="0.15476 -${0.140618} -${0.026643 + 0.014}"
+      rpy="-${M_PI/2} ${M_PI/2} 0" />
+    <!--<origin
       xyz="0.15476 -${0.020382 + 0.161} -${0.026643 + 0.014}"
-      rpy="${M_PI/2} -${M_PI/2} 0" />
+      rpy="-${M_PI/2} ${M_PI/2} 0" />-->
     <origin
       xyz="0.0536535102814494 -0.00979339452125411 0.0186240655062149"
@@ -69,5 +104,5 @@
     <origin
       xyz="0.15476 ${0.020382 + 0.161} -${0.026643 + 0.014}"
-      rpy="-${M_PI/2} -${M_PI/2} 0" />
+      rpy="-${M_PI/2} ${M_PI/2} 0" />
     <origin
       xyz="0.0536535102814494 0.00979339452125411 0.0186240655062149"

File: panther_description/urdf/sprocket.urdf.xacro (robot description, xacro)
@@ -30,5 +30,5 @@
     <axis xyz="0 0 -1" />
     <limit effort="12" velocity="22"/>
-    <joint_properties damping="0.0" friction="0.0"/>
+    <joint_properties damping="1.0" friction="1.0"/>
   </joint>
   <transmission name="${name}_trans" type="SimpleTransmission">
@@ -38,5 +38,5 @@
     </actuator>
     <joint name="${name}">
-      <hardwareInterface>VelocityJointInterface</hardwareInterface>
+      <hardwareInterface>hardware_interface/VelocityJointInterface</hardwareInterface>
     </joint>
   </transmission>

File: panther_description/urdf/track.urdf.xacro (robot description, xacro)
@@ -1,3 +1,28 @@
 <?xml version="1.0"?>
+<!--
+Copyright (C) 2017, Raffaello Bonghi <raffaello@rnext.it>
+All rights reserved
+Redistribution and use in source and binary forms, with or without
+modification, are permitted provided that the following conditions are met:
+1. Redistributions of source code must retain the above copyright
+   notice, this list of conditions and the following disclaimer.
+2. Redistributions in binary form must reproduce the above copyright
+   notice, this list of conditions and the following disclaimer in the
+   documentation and/or other materials provided with the distribution.
+3. Neither the name of the copyright holder nor the names of its
+   contributors may be used to endorse or promote products derived
+   from this software without specific prior written permission.
+THIS SOFTWARE IS PROVIDED BY THE COPYRIGHT HOLDERS AND
+CONTRIBUTORS "AS IS" AND ANY EXPRESS OR IMPLIED WARRANTIES, INCLUDING,
+BUT NOT LIMITED TO, THE IMPLIED WARRANTIES OF MERCHANTABILITY AND FITNESS
+FOR A PARTICULAR PURPOSE ARE DISCLAIMED. IN NO EVENT SHALL THE COPYRIGHT
+HOLDER OR CONTRIBUTORS BE LIABLE FOR ANY DIRECT, INDIRECT, INCIDENTAL,
+SPECIAL, EXEMPLARY, OR CONSEQUENTIAL DAMAGES (INCLUDING, BUT NOT LIMITED TO,
+PROCUREMENT OF SUBSTITUTE GOODS OR SERVICES; LOSS OF USE, DATA, OR PROFITS;
+OR BUSINESS INTERRUPTION) HOWEVER CAUSED AND ON ANY THEORY OF LIABILITY,
+WHETHER IN CONTRACT, STRICT LIABILITY, OR TORT (INCLUDING NEGLIGENCE
+OR OTHERWISE) ARISING IN ANY WAY OUT OF THE USE OF THIS SOFTWARE,
+EVEN IF ADVISED OF THE POSSIBILITY OF SUCH DAMAGE.
+-->
 <robot xmlns:xacro="http://ros.org/wiki/xacro" name="track">
  <!-- passive_wheel_type tye: (1) continuous or (2) fixed -->

Commit message: Added ZED camera and solve some errors

File: panther_description/urdf/panther.urdf.xacro (robot description, xacro)
@@ -71,5 +71,5 @@
   <!-- ZED -->
   <xacro:zedcamera parent="frame_link">
-    <origin xyz="-0.03600 0 0.1900" rpy="${M_PI} ${M_PI} ${-M_PI/2}" />
+    <origin xyz="-0.03600 0 0.1700" rpy="0 0 0" />
   </xacro:zedcamera>
   <!-- ZED - END -->

File: panther_description/urdf/zedcamera.urdf.xacro (robot description, xacro)
@@ -30,4 +30,90 @@
   <xacro:macro name="zedcamera" params="parent *joint_pose">
   <link name="zed_stand_link">
+    <inertial>
+      <origin xyz="0 -0.0184 0.0173" rpy="0 0 0" />
+      <mass value="0.0173" />
+      <inertia ixx="2.76959607332778E-06" ixy="-7.16716953193216E-11" ixz="-1.34923517166624E-10"
+                                          iyy="6.44872593702919E-06"  iyz="6.78675778442728E-08"
+                                                                      izz="4.02458373877404E-06" />
+    </inertial>
+    <visual>
+      <origin xyz="0 0 0.02" rpy="0 0 ${M_PI/2}" />
+      <geometry>
+        <mesh filename="${path_meshes}/zed/stand_link.STL" />
+      </geometry>
+      <material name="Black" />
+    </visual>
+  </link>
+  <joint name="zed_stand_sensor" type="fixed">
+    <xacro:insert_block name="joint_pose"/>
+    <parent link="${parent}" />
+    <child link="zed_stand_link" />
+    <axis xyz="0 0 0" />
+  </joint>
+  <link name="zed_camera_link">
+    <visual>
+      <origin xyz="0 0 0" rpy="0 0 0"/>
+      <geometry>
+        <mesh filename="package://zed_wrapper/urdf/ZED.stl" />
+      </geometry>
+      <material name="light_grey">
+        <color rgba="0.8 0.8 0.8 0.95"/>
+      </material>
+    </visual>
+  </link>
+  <joint name="zed_camera_joint" type="fixed">
+    <origin xyz="0.0165 0 0.02" rpy="0 0 0" />
+    <parent link="zed_stand_link" />
+    <child link="zed_camera_link" />
+    <axis xyz="0 0 0" />
+  </joint>
+  <link name="zed_initial_frame" />
+  <joint name="zed_initial_joint" type="fixed">
+    <origin xyz="0 0.06 0" rpy="0 0 0" />
+    <parent link="zed_camera_link" />
+    <child link="zed_initial_frame" />
+    <axis xyz="0 0 0" />
+  </joint>
+  <link name="zed_depth_frame" />
+  <joint name="zed_depth_joint" type="fixed">
+    <origin xyz="0 0.0 0" rpy="-${M_PI/2} 0 -${M_PI/2}" />
+    <parent link="zed_initial_frame" />
+    <child link="zed_depth_frame" />
+    <axis xyz="0 0 0" />
+  </joint>
+  <link name="ZED_left_camera">
+     <visual>
+       <origin xyz="0 0 0" rpy="0 1.57 0"/>
+       <geometry>
+         <cylinder radius="0.007" length=".031"/>
+       </geometry>
+       <material name="dark_grey">
+         <color rgba="0.1 0.1 0.1 1"/>
+       </material>
+     </visual>
+  </link>
+  <link name="ZED_right_camera">
+     <visual>
+       <origin xyz="0 0 0" rpy="0 1.57 0"/>
+       <geometry>
+         <cylinder radius="0.007" length=".031"/>
+       </geometry>
+       <material name="dark_grey">
+         <color rgba="0.1 0.1 0.1 1"/>
+       </material>
+     </visual>
+  </link>
+  <joint name="ZED_left_camera_joint" type="fixed">
+    <origin xyz="0 0 0" rpy="0 0 0" />
+    <parent link="zed_initial_frame" />
+    <child link="ZED_left_camera" />
+    <axis xyz="0 0 0" />
+  </joint>
+  <joint name="ZED_right_camera_joint" type="fixed">
+      <parent link="ZED_left_camera"/>
+      <child link="ZED_right_camera"/>
+      <origin xyz="0 -0.12 0" rpy="0 0 0" />
+  </joint>
+<!--  <link name="zed_stand_link">
     <inertial>
       <origin xyz="0 -0.0184 0.0173" rpy="0 0 0" />
@@ -96,5 +182,5 @@
       <child link="zed_right_optical_frame" />
     </joint>
-    <link name="zed_right_optical_frame"/>
+    <link name="zed_right_optical_frame"/>-->
   </xacro:macro>
 </robot>

Commit message: Added lidar in panther description

File: panther_description/urdf/panther.urdf.xacro (robot description, xacro)
@@ -30,5 +30,5 @@
   <xacro:include filename="$(find panther_description)/urdf/chassis.urdf.xacro" />
   <xacro:include filename="$(find panther_description)/urdf/track.urdf.xacro" />
-  <xacro:include filename="$(find panther_description)/urdf/zedcamera.urdf.xacro" />
+  <xacro:include filename="$(find panther_description)/urdf/zed_lidar.urdf.xacro" />
   <xacro:include filename="$(find panther_description)/urdf/imu.urdf.xacro" />
   <!-- Included URDF/XACRO Files -->
@@ -70,7 +70,7 @@
   <!-- Chassis - END -->
   <!-- ZED -->
-  <xacro:zedcamera parent="frame_link">
+  <xacro:zed_lidar parent="frame_link">
     <origin xyz="-0.03600 0 0.1700" rpy="0 0 0" />
-  </xacro:zedcamera>
+  </xacro:zed_lidar>
   <!-- ZED - END -->
   <!-- IMU -->

File: panther_description/urdf/zed_lidar.urdf.xacro (robot description, xacro)
@@ -25,9 +25,9 @@
 EVEN IF ADVISED OF THE POSSIBILITY OF SUCH DAMAGE.
 -->
-<robot name="zedcamera" xmlns:xacro="http://ros.org/wiki/xacro">
+<robot name="zed_lidar" xmlns:xacro="http://ros.org/wiki/xacro">
 <xacro:property name="optical_y_offset" value="0.06" />
 <xacro:property name="optical_x_offset" value="0.03" />
-  <xacro:macro name="zedcamera" params="parent *joint_pose">
-  <link name="zed_stand_link">
+  <xacro:macro name="zed_lidar" params="parent *joint_pose">
+  <link name="stand_link">
     <inertial>
       <origin xyz="0 -0.0184 0.0173" rpy="0 0 0" />
@@ -38,17 +38,48 @@
     </inertial>
     <visual>
-      <origin xyz="0 0 0.02" rpy="0 0 ${M_PI/2}" />
+      <origin xyz="-0.029 0 -0.0038" rpy="${M_PI/2} 0 ${M_PI}" />
       <geometry>
-        <mesh filename="${path_meshes}/zed/stand_link.STL" />
+        <mesh filename="${path_meshes}/zed-lidar-stand/stand_link.STL" />
       </geometry>
       <material name="Black" />
     </visual>
   </link>
-  <joint name="zed_stand_sensor" type="fixed">
+  <joint name="stand_sensor" type="fixed">
     <xacro:insert_block name="joint_pose"/>
     <parent link="${parent}" />
-    <child link="zed_stand_link" />
+    <child link="stand_link" />
     <axis xyz="0 0 0" />
   </joint>
+  <!-- Laser -->
+  <link name="laser_link">
+    <inertial>
+      <origin xyz="0 -0.0184 0.0173" rpy="0 0 0" />
+      <mass value="0.0173" />
+      <inertia ixx="2.76959607332778E-06" ixy="-7.16716953193216E-11" ixz="-1.34923517166624E-10"
+                                          iyy="6.44872593702919E-06"  iyz="6.78675778442728E-08"
+                                                                      izz="4.02458373877404E-06" />
+    </inertial>
+    <visual>
+      <origin xyz="-0.005 -0.075 -0.012" rpy="0 0 ${M_PI}" />
+      <geometry>
+        <mesh filename="${path_meshes}/lidar/rplidar_link.STL" />
+      </geometry>
+      <material name="DarkGrey" />
+    </visual>
+  </link>
+  <joint name="laser_sensor_base" type="fixed">
+    <origin xyz="-0.03 0 0.02" rpy="0 0 0" />
+    <parent link="stand_link" />
+    <child link="laser_link" />
+    <axis xyz="0 0 0" />
+  </joint>
+  <link name="laser_frame" />
+  <joint name="laser_sensor" type="fixed">
+    <origin xyz="0 0 0.027" rpy="0 0 0" />
+    <parent link="laser_link" />
+    <child link="laser_frame" />
+    <axis xyz="0 0 0" />
+  </joint>
+  <!-- ZED camera -->
   <link name="zed_camera_link">
     <visual>
@@ -63,6 +94,6 @@
   </link>
   <joint name="zed_camera_joint" type="fixed">
-    <origin xyz="0.0165 0 0.02" rpy="0 0 0" />
-    <parent link="zed_stand_link" />
+    <origin xyz="0.028 0 0.021" rpy="0 0 0" />
+    <parent link="stand_link" />
     <child link="zed_camera_link" />
     <axis xyz="0 0 0" />

Commit message: Refactoring urdf and load ZED from zed package

File: panther_description/urdf/panther.urdf.xacro (robot description, xacro)
@@ -29,7 +29,8 @@
   <xacro:include filename="$(find panther_description)/urdf/materials.urdf" />
   <xacro:include filename="$(find panther_description)/urdf/chassis.urdf.xacro" />
-  <xacro:include filename="$(find panther_description)/urdf/track.urdf.xacro" />
+  <xacro:include filename="$(find panther_description)/urdf/track/track.urdf.xacro" />
   <xacro:include filename="$(find panther_description)/urdf/zed_lidar.urdf.xacro" />
   <xacro:include filename="$(find panther_description)/urdf/imu.urdf.xacro" />
+  <xacro:include filename="$(find zed_wrapper)/urdf/zed.urdf.xacro" /> <!-- ZED external xacro -->
   <!-- Included URDF/XACRO Files -->
   <!-- Global properties -->
@@ -65,4 +66,7 @@
     <origin xyz="-0.03600 0 0.1700" rpy="0 0 0" />
   </xacro:zed_lidar>
+  <xacro:zed parent="stand_link" camera_name="zed" camera_model="zed2">
+    <origin xyz="0.028 0 0.021" rpy="0 0 0" />
+  </xacro:zed>
   <!-- ZED - END -->
   <!-- IMU -->

File: panther_description/urdf/track/track.urdf.xacro (robot description, xacro)
@@ -1,5 +1,5 @@
 <?xml version="1.0"?>
 <!--
-Copyright (C) 2017, Raffaello Bonghi <raffaello@rnext.it>
+Copyright (C) 2020, Raffaello Bonghi <raffaello@rnext.it>
 All rights reserved
 Redistribution and use in source and binary forms, with or without
@@ -26,7 +26,7 @@
 -->
 <robot xmlns:xacro="http://ros.org/wiki/xacro" name="track">
-  <xacro:include filename="$(find panther_description)/urdf/sprocket.urdf.xacro" />
-  <xacro:include filename="$(find panther_description)/urdf/gear.urdf.xacro" />
-  <xacro:include filename="$(find panther_description)/urdf/wheel.urdf.xacro" />
+  <xacro:include filename="$(find panther_description)/urdf/track/sprocket.urdf.xacro" />
+  <xacro:include filename="$(find panther_description)/urdf/track/gear.urdf.xacro" />
+  <xacro:include filename="$(find panther_description)/urdf/track/wheel.urdf.xacro" />
   <xacro:macro name="track" params="type parent">
   <!-- Define orientation -->

File: panther_description/urdf/zed_lidar.urdf.xacro (robot description, xacro)
@@ -82,5 +82,5 @@
   </joint>
   <!-- ZED camera -->
-    <link name="zed_center">
+  <!--  <link name="zed_center">
     <visual>
         <origin xyz="0 0 0" rpy="0 0 0"/>
@@ -136,5 +136,5 @@
         <child link="zed_right_camera"/>
         <origin xyz="0 -0.06 0" rpy="0 0 0" />
-    </joint>
+    </joint> -->
   </xacro:macro>
 </robot>
