Commit message: Refactoring Panther urdf

File: panther_description/urdf/panther.urdf.xacro (robot description, xacro)
@@ -26,56 +26,52 @@
 -->
 <robot name="panther" xmlns:xacro="http://ros.org/wiki/xacro">
-  <!-- Included URDF/XACRO Files -->
-  <xacro:include filename="$(find panther_description)/urdf/materials.urdf" />
-  <xacro:include filename="$(find panther_description)/urdf/chassis.urdf.xacro" />
-  <xacro:include filename="$(find panther_description)/urdf/track/track.urdf.xacro" />
-  <xacro:include filename="$(find panther_description)/urdf/zed_lidar.urdf.xacro" />
-  <xacro:include filename="$(find panther_description)/urdf/imu.urdf.xacro" />
-  <xacro:include filename="$(find zed_wrapper)/urdf/zed.urdf.xacro" /> <!-- ZED external xacro -->
-  <!-- Included URDF/XACRO Files -->
-  <!-- Global properties -->
-  <xacro:property name="path_meshes" value="package://panther_description/meshes"/>
-  <xacro:property name="M_PI" value="3.14159"/>
-  <!-- Global properties -->
-  <!-- Sprocket and gear properties -->
-  <xacro:property name="sprocket_radius" value="0.0325"/>
-  <xacro:property name="sprocket_leght" value="0.05"/>
-  <xacro:property name="sprocket_teeth" value="24"/>
-  <xacro:property name="gear_teeth" value="16"/>
-  <xacro:property name="wheel_offset_x" value="-0.00"/>
-  <xacro:property name="wheel_offset_y" value="0.08"/>
-  <xacro:property name="wheel_offset_z" value="${wheel_radius}"/>
-  <!-- Sprocket and gear properties -->
-  <!-- base_link -->
-  <link name="base_link">
-    <visual>
-      <origin xyz="0 0 0" rpy="0 0 0" />
-      <geometry>
-        <cylinder length="0.001" radius="0.05"/>
-      </geometry>
-      <material name="Green" />
-    </visual>
-  </link>
-  <!-- Chassis -->
-  <xacro:chassis parent="base_link">
-    <origin xyz="0 0 0.08" rpy="0 0 0" />
-  </xacro:chassis>
-  <!-- Chassis - END -->
-  <!-- ZED -->
-  <xacro:zed_lidar parent="frame_link">
-    <origin xyz="-0.03600 0 0.1700" rpy="0 0 0" />
-  </xacro:zed_lidar>
-  <xacro:zed parent="stand_link" camera_name="zed" camera_model="zed2">
-    <origin xyz="0.028 0 0.021" rpy="0 0 0" />
-  </xacro:zed>
-  <!-- ZED - END -->
-  <!-- IMU -->
-  <xacro:imu parent="frame_link">
-    <origin xyz="-0.0420817256507905 0 0.091441320597534" rpy="0 ${M_PI/2} 0" />
-  </xacro:imu>
-  <!-- IMU -->
-  <!-- Track -->
-  <xacro:track type="left" parent="frame_link" />
-  <xacro:track type="right" parent="frame_link" />
-  <!-- Track - END -->
+    <xacro:include filename="$(find panther_description)/urdf/materials.urdf" />
+    <!-- Panther parts -->
+    <xacro:include filename="$(find panther_description)/urdf/chassis/chassis.urdf.xacro" />
+    <xacro:include filename="$(find panther_description)/urdf/chassis/stand.urdf.xacro" />
+    <xacro:include filename="$(find panther_description)/urdf/track/track.urdf.xacro" />
+    <!-- Sensors -->
+    <xacro:include filename="$(find panther_description)/urdf/sensors/imu.urdf.xacro" />
+    <xacro:include filename="$(find panther_description)/urdf/sensors/rplidar.urdf.xacro" />
+    <xacro:include filename="$(find zed_wrapper)/urdf/zed.urdf.xacro" /> <!-- ZED external xacro -->
+    <!-- Arguments -->
+    <xacro:arg name="zed_model"   default="zed2" />
+    <!-- Global properties -->
+    <xacro:property name="path_meshes" value="package://panther_description/meshes"/>
+    <xacro:property name="M_PI" value="3.14159"/>
+    <!-- Sprocket and gear properties -->
+    <xacro:property name="sprocket_radius" value="0.0325"/>
+    <xacro:property name="sprocket_leght"  value="0.05"/>
+    <xacro:property name="sprocket_teeth"  value="24"/>
+    <xacro:property name="gear_teeth"      value="16"/>
+    <xacro:property name="wheel_offset_x"  value="-0.00"/>
+    <xacro:property name="wheel_offset_y"  value="0.08"/>
+    <xacro:property name="wheel_offset_z"  value="${wheel_radius}"/>
+    <!-- base_link -->
+    <link name="base_link">
+        <visual>
+            <origin xyz="0 0 0" rpy="0 0 0" />
+            <geometry><cylinder length="0.001" radius="0.05"/></geometry>
+            <material name="Green" />
+        </visual>
+    </link>
+    <!-- Panther body -->
+    <xacro:chassis parent="base_link">
+        <origin xyz="0 0 0.08" rpy="0 0 0" />
+    </xacro:chassis>
+    <xacro:track type="left" parent="frame_link" />
+    <xacro:track type="right" parent="frame_link" />
+    <xacro:stand parent="frame_link" model="stand_rplidar_zed">
+        <origin xyz="-0.03600 0 0.1700" rpy="0 0 0" />
+    </xacro:stand>
+    <!-- Sensors -->
+    <xacro:razor_imu parent="frame_link">
+        <origin xyz="-0.0420817256507905 0 0.091441320597534" rpy="0 ${M_PI/2} 0" />
+    </xacro:razor_imu>
+    <xacro:zed parent="stand_link" camera_name="zed" camera_model="$(arg zed_model)">
+        <origin xyz="0.028 0 0.021" rpy="0 0 0" />
+    </xacro:zed>
+    <xacro:rplidar parent="stand_link">
+        <origin xyz="-0.03 0 0.02" rpy="0 0 0" />
+    </xacro:rplidar>
 </robot>

File: panther_description/urdf/sensors/rplidar.urdf.xacro (robot description, xacro)
@@ -25,35 +25,36 @@
 EVEN IF ADVISED OF THE POSSIBILITY OF SUCH DAMAGE.
 -->
-<robot xmlns:xacro="http://ros.org/wiki/xacro" name="imu">
-  <xacro:macro name="imu" params="parent *joint_pose">
-    <link name="imu_board_link">
-      <inertial>
-        <origin xyz="0.0002 0.003 -0.00025" rpy="0 0 0" />
-        <mass value="0.0045" />
-        <inertia
-          ixx="6.80127923442653E-07" ixy="2.58853590724977E-08" ixz="6.27330058259111E-09"
-                                     iyy="2.67621227004883E-07" iyz="3.00971478682596E-08"
-                                                                izz="9.29933868272119E-07" />
-      </inertial>
-      <visual>
-        <origin xyz="0 0 0" rpy="0 0 0" />
-        <geometry>
-          <mesh filename="${path_meshes}/imu/imu_Link.STL" />
-        </geometry>
-        <material name="Red" />
-      </visual>
-    </link>
-    <joint name="imu_board_joint" type="fixed">
-      <xacro:insert_block name="joint_pose"/>
-      <parent link="${parent}" />
-      <child link="imu_board_link" />
-    </joint>
-    <!-- Required "base_imu_link" to read the razor IMU data -->
-    <link name="base_imu_link" />
-    <joint name="base_imu_joint" type="fixed">
-      <origin xyz="0 0 0" rpy="0 ${-M_PI/2} 0" />
-      <parent link="imu_board_link" />
-      <child link="base_imu_link" />
-    </joint>
- </xacro:macro>
+<robot name="rplidar" xmlns:xacro="http://ros.org/wiki/xacro">
+    <xacro:macro name="rplidar" params="parent *joint_pose">
+        <!-- Laser -->
+        <link name="laser_link">
+            <inertial>
+                <origin xyz="0 -0.0184 0.0173" rpy="0 0 0" />
+                <mass value="0.0173" />
+                <inertia ixx="2.77E-06" ixy="-7.17E-11" ixz="-1.35E-10"
+                         iyy="6.45E-06" iyz="6.79E-08"
+                                                        izz="4.02E-06" />
+                </inertial>
+            <visual>
+                <origin xyz="-0.005 -0.075 -0.012" rpy="0 0 ${M_PI}" />
+                <geometry>
+                    <mesh filename="${path_meshes}/sensors/rplidar.stl" />
+                </geometry>
+                <material name="DarkGrey" />
+            </visual>
+        </link>
+        <joint name="laser_sensor_base" type="fixed">
+            <xacro:insert_block name="joint_pose"/>
+            <parent link="${parent}" />
+            <child link="laser_link" />
+            <axis xyz="0 0 0" />
+        </joint>
+        <link name="laser_frame" />
+        <joint name="laser_sensor" type="fixed">
+            <origin xyz="0 0 0.027" rpy="0 0 ${M_PI}" />
+            <parent link="laser_link" />
+            <child link="laser_frame" />
+            <axis xyz="0 0 0" />
+        </joint>
+    </xacro:macro>
 </robot>

Commit message: Add ultrasounds

File: panther_description/urdf/panther.urdf.xacro (robot description, xacro)
@@ -33,4 +33,5 @@
     <xacro:include filename="$(find panther_description)/urdf/track/track.urdf.xacro" />
     <!-- Sensors -->
+    <xacro:include filename="$(find panther_description)/urdf/sensors/ultrasounds.urdf.xacro" />
     <xacro:include filename="$(find panther_description)/urdf/sensors/imu.urdf.xacro" />
     <xacro:include filename="$(find panther_description)/urdf/sensors/rplidar.urdf.xacro" />
@@ -82,4 +83,13 @@
     </xacro:if>
     <!-- Sensors -->
+    <xacro:ultrasounds name="SFR10_left" parent="frame_link">
+        <origin xyz="0.15 0.095 -0.015" rpy="0 0 0" />
+    </xacro:ultrasounds>
+    <xacro:ultrasounds name="SFR10_right" parent="frame_link">
+        <origin xyz="0.15 -0.095 -0.015" rpy="0 0 0" />
+    </xacro:ultrasounds>
+    <xacro:ultrasounds name="SFR10_rear" parent="frame_link">
+        <origin xyz="-0.15 0 -0.015" rpy="${M_PI} ${M_PI} 0" />
+    </xacro:ultrasounds>
     <xacro:razor_imu parent="frame_link">
         <origin xyz="-0.0420817256507905 0 0.091441320597534" rpy="0 ${M_PI/2} 0" />

File: panther_description/urdf/sensors/ultrasounds.urdf.xacro (robot description, xacro)
@@ -25,33 +25,19 @@
 EVEN IF ADVISED OF THE POSSIBILITY OF SUCH DAMAGE.
 -->
-<robot xmlns:xacro="http://ros.org/wiki/xacro" name="razor_imu">
-    <xacro:macro name="razor_imu" params="parent *joint_pose">
-        <link name="imu_board_link">
-            <inertial>
-                <origin xyz="0.0002 0.003 -0.00025" rpy="0 0 0" />
-                <mass value="0.0045" />
-                <inertia ixx="6.80E-07" ixy="2.59E-08" ixz="6.27E-09"
-                         iyy="2.68E-07" iyz="3.01E-08"
-                                                       izz="9.30E-07" />
-            </inertial>
+<robot xmlns:xacro="http://ros.org/wiki/xacro" name="ultrasounds">
+    <xacro:macro name="ultrasounds" params="name parent *joint_pose">
+        <link name="${name}_frame">
             <visual>
                 <origin xyz="0 0 0" rpy="0 0 0" />
                 <geometry>
-                    <mesh filename="${path_meshes}/sensors/razor_imu.stl" />
+                    <box size="0.03 0.03 0.015"/>
                 </geometry>
-                <material name="Red" />
+                <material name="Black" />
             </visual>
         </link>
-        <joint name="imu_board_joint" type="fixed">
+        <joint name="${name}_joint" type="fixed">
             <xacro:insert_block name="joint_pose"/>
             <parent link="${parent}" />
-            <child link="imu_board_link" />
-        </joint>
-        <!-- Required "base_imu_link" to read the razor IMU data -->
-        <link name="base_imu_link" />
-        <joint name="base_imu_joint" type="fixed">
-            <origin xyz="0 0 0" rpy="0 ${-M_PI/2} 0" />
-            <parent link="imu_board_link" />
-            <child link="base_imu_link" />
+            <child link="${name}_frame" />
         </joint>
     </xacro:macro>
