Commit message: Refactoring Panther urdf adding arguments option for boards

File: panther_description/urdf/chassis/chassis.urdf.xacro (robot description, xacro)
@@ -189,112 +189,4 @@
     <axis xyz="0 0 0" />
   </joint>
-  <link name="ssd_link">
-    <inertial>
-      <origin xyz="0.00095 -0.00011 0.0031" rpy="0 0 0" />
-      <mass value="0.0427" />
-      <inertia ixx="1.77491831386846E-05" ixy="2.28450378389574E-07" ixz="-1.93475819680817E-08"
-        iyy="3.5077947505707E-05" iyz="2.31216416056502E-09"
-        izz="5.2544572820951E-05" />
-    </inertial>
-    <visual>
-      <origin xyz="0 0 0" rpy="0 0 0" />
-      <geometry>
-        <mesh filename="${path_meshes}/chassis/ssd_link.STL" />
-      </geometry>
-      <material name="Grey" />
-    </visual>
-  </link>
-  <joint name="ssd_joint" type="fixed">
-    <origin
-      xyz="0.0465 0.03075 0.04674"
-      rpy="${M_PI} 0 ${M_PI}" />
-    <parent link="frame_link" />
-    <child link="ssd_link" />
-    <axis xyz="0 0 0" />
-  </joint>
-  <link name="jetson_carrier_link">
-    <inertial>
-      <origin xyz="0.0385 0.02167 0.00953" rpy="0 0 0" />
-      <mass value="0.05208" />
-      <inertia ixx="1.36170018377782E-05" ixy="8.38611240500124E-07" ixz="-4.79467802124809E-07"
-        iyy="3.618139427206E-05" iyz="-5.02791911288937E-07"
-        izz="4.27350235788097E-05" />
-    </inertial>
-    <visual>
-      <origin xyz="0 0 0" rpy="0 0 0" />
-      <geometry>
-        <mesh filename="${path_meshes}/chassis/jetson/carrier_link.STL" />
-      </geometry>
-      <material name="DarkGrey" />
-    </visual>
-  </link>
-  <joint name="jetson_carrier_joint" type="fixed">
-    <origin
-      xyz="0.1 0.01 0.055"
-      rpy="${-M_PI/2} 0 ${M_PI}" />
-    <parent link="frame_link" />
-    <child link="jetson_carrier_link" />
-    <axis xyz="0 0 0" />
-  </joint>
-  <link name="jetson_tx1_link">
-    <inertial>
-      <origin xyz="0.0339 -0.0064 -0.00574" rpy="0 0 0" />
-      <mass value="0.0747" />
-      <inertia ixx="0.000189260214606175" ixy="-3.62601702140744E-06" ixz="1.04156349484491E-06"
-        iyy="0.000194645180332423" iyz="5.44491260645182E-08"
-        izz="0.000382161755658342" />
-    </inertial>
-    <visual>
-      <origin xyz="0 0 0" rpy="0 0 0" />
-      <geometry>
-        <mesh filename="${path_meshes}/chassis/jetson/tx1_core_link.STL" />
-      </geometry>
-      <material name="GunMetalGrey" />
-    </visual>
-  </link>
-  <joint name="jetson_tx1_joint" type="fixed">
-    <origin xyz="0 0 0" rpy="0 0 0" />
-    <parent link="jetson_carrier_link" />
-    <child link="jetson_tx1_link" />
-    <axis xyz="0 0 0" />
-  </joint>
-  <link name="battery_link">
-    <inertial>
-      <origin xyz="0 0 0.018" rpy="0 0 0" />
-      <mass value="0.24981" />
-      <inertia
-        ixx="0.00044483" ixy="1.2332E-20" ixz="1.0603E-21"
-        iyy="7.6356E-05" iyz="2.4007E-20"
-        izz="0.00046843" />
-    </inertial>
-    <visual>
-      <origin xyz="0 0 0" rpy="0 0 0" />
-      <geometry>
-        <mesh filename="${path_meshes}/chassis/battery_link.STL" />
-      </geometry>
-      <material name="Blue" />
-    </visual>
-  </link>
-  <joint name="battery_joint" type="fixed">
-    <origin xyz="-0.13 0 0.01" rpy="0 0 0" />
-    <parent link="frame_link" />
-    <child link="battery_link" />
-    <axis xyz="0 0 0" />
-  </joint>
-  <link name="unav_link">
-    <visual>
-      <origin xyz="0 0 0" rpy="0 0 0" />
-      <geometry>
-        <box size="0.09 0.09 0.005"/>
-      </geometry>
-      <material name="Blue" />
-    </visual>
-  </link>
-  <joint name="unav_joint" type="fixed">
-    <origin xyz="-0.10 0 0.13" rpy="0 0 0" />
-    <parent link="frame_link" />
-    <child link="unav_link" />
-    <axis xyz="0 0 0" />
-  </joint>
   </xacro:macro>
 </robot>

File: panther_description/urdf/panther.urdf.xacro (robot description, xacro)
@@ -30,4 +30,5 @@
     <xacro:include filename="$(find panther_description)/urdf/chassis/chassis.urdf.xacro" />
     <xacro:include filename="$(find panther_description)/urdf/chassis/stand.urdf.xacro" />
+    <xacro:include filename="$(find panther_description)/urdf/chassis/battery.urdf.xacro" />
     <xacro:include filename="$(find panther_description)/urdf/track/track.urdf.xacro" />
     <!-- Sensors -->
@@ -35,6 +36,11 @@
     <xacro:include filename="$(find panther_description)/urdf/sensors/rplidar.urdf.xacro" />
     <xacro:include filename="$(find zed_wrapper)/urdf/zed.urdf.xacro" /> <!-- ZED external xacro -->
+    <!-- Boards -->
+    <xacro:include filename="$(find panther_description)/urdf/boards/jetson.urdf.xacro" />
     <!-- Arguments -->
-    <xacro:arg name="zed_model"   default="zed2" />
+    <xacro:arg name="zed_model"   default="zed2"/> <!-- Follow zed_repository -->
+    <xacro:arg name="jetson"      default="xavier"/> <!-- options: tx, xavier -->
+    <xacro:arg name="motor_board" default="roboteq"/> <!-- options: unav, roboteq -->
+    <xacro:arg name="ssd"         default="false"/>
     <!-- Global properties -->
     <xacro:property name="path_meshes" value="package://panther_description/meshes"/>
@@ -48,4 +54,5 @@
     <xacro:property name="wheel_offset_y"  value="0.08"/>
     <xacro:property name="wheel_offset_z"  value="${wheel_radius}"/>
+    <xacro:property name="mboard" value="$(arg motor_board)"/>
     <!-- base_link -->
     <link name="base_link">
@@ -65,4 +72,13 @@
         <origin xyz="-0.03600 0 0.1700" rpy="0 0 0" />
     </xacro:stand>
+    <xacro:battery parent="frame_link" mass="0.24981">
+        <origin xyz="-0.13 0 0.01" rpy="0 0 0" />
+    </xacro:battery>
+    <xacro:if value="$(arg ssd)">
+        <xacro:include filename="$(find panther_description)/urdf/chassis/ssd.urdf.xacro" />
+        <xacro:ssd parent="frame_link">
+            <origin xyz="0.0465 0.03075 0.04674" rpy="${M_PI} 0 ${M_PI}" />
+        </xacro:ssd>
+    </xacro:if>
     <!-- Sensors -->
     <xacro:razor_imu parent="frame_link">
@@ -75,3 +91,19 @@
         <origin xyz="-0.03 0 0.02" rpy="0 0 0" />
     </xacro:rplidar>
+    <!-- Boards -->
+    <xacro:jetson parent="frame_link" model="$(arg jetson)">
+        <origin xyz="0.08 0 0.05" rpy="0 0 0" />
+    </xacro:jetson>
+    <xacro:if value="${mboard == 'unav'}">
+        <xacro:include filename="$(find panther_description)/urdf/boards/unav.urdf.xacro" />
+        <xacro:unav parent="frame_link">
+            <origin xyz="-0.10 0 0.12" rpy="0 0 0" />
+        </xacro:unav>
+    </xacro:if>
+    <xacro:if value="${mboard == 'roboteq'}">
+        <xacro:include filename="$(find panther_description)/urdf/boards/roboteq.urdf.xacro" />
+        <xacro:roboteq parent="frame_link">
+            <origin xyz="-0.11 0 0.12" rpy="0 0 0" />
+        </xacro:roboteq>
+    </xacro:if>
 </robot>
