Commit message: Enable/Disable ultrasounds. Rearrange URDF for https://github.com/rpanther/panther_simulation/issues/1

File: panther_description/urdf/boards/jetson.urdf.xacro (robot description, xacro)
@@ -35,7 +35,8 @@
             <link name="jetson_carrier_link">
                 <visual>
-                    <origin xyz="0 0 0.025" rpy="0 0 0" />
+                    <origin xyz="-0.047 0.048 0.011" rpy="${-M_PI/2} 0 ${-M_PI/2}" />
                     <geometry>
-                        <box size="0.12 0.12 0.05" />
+                        <!--<box size="0.12 0.12 0.05" />-->
+                        <mesh filename="${path_meshes}/boards/xavier_link.stl"/>
                     </geometry>
                     <material name="Black" />

File: panther_description/urdf/chassis/chassis.urdf.xacro (robot description, xacro)
@@ -87,5 +87,5 @@
     </inertial>
     <visual>
-      <origin xyz="0 0 0" rpy="0 0 ${M_PI}" />
+      <origin xyz="0 0 0.0788" rpy="0 0 ${M_PI}" />
       <geometry>
         <mesh filename="${path_meshes}/chassis/cover_link.STL" />

File: panther_description/urdf/panther.urdf.xacro (robot description, xacro)
@@ -26,94 +26,16 @@
 -->
 <robot name="panther" xmlns:xacro="http://ros.org/wiki/xacro">
-    <xacro:include filename="$(find panther_description)/urdf/materials.urdf" />
-    <!-- Panther parts -->
-    <xacro:include filename="$(find panther_description)/urdf/chassis/chassis.urdf.xacro" />
-    <xacro:include filename="$(find panther_description)/urdf/chassis/stand.urdf.xacro" />
-    <xacro:include filename="$(find panther_description)/urdf/chassis/battery.urdf.xacro" />
-    <xacro:include filename="$(find panther_description)/urdf/track/track.urdf.xacro" />
-    <!-- Sensors -->
-    <xacro:include filename="$(find panther_description)/urdf/sensors/ultrasounds.urdf.xacro" />
-    <xacro:include filename="$(find panther_description)/urdf/sensors/imu.urdf.xacro" />
-    <xacro:include filename="$(find panther_description)/urdf/sensors/rplidar.urdf.xacro" />
-    <xacro:include filename="$(find zed_wrapper)/urdf/zed.urdf.xacro" /> <!-- ZED external xacro -->
-    <!-- Boards -->
-    <xacro:include filename="$(find panther_description)/urdf/boards/jetson.urdf.xacro" />
+   <xacro:include filename="$(find panther_description)/urdf/robot.urdf.xacro" />
     <!-- Arguments -->
-    <xacro:arg name="zed_model"   default="zed2"/> <!-- Follow zed_repository -->
-    <xacro:arg name="jetson"      default="xavier"/> <!-- options: tx, xavier -->
-    <xacro:arg name="motor_board" default="roboteq"/> <!-- options: unav, roboteq -->
-    <xacro:arg name="ssd"         default="false"/>
-    <!-- Global properties -->
-    <xacro:property name="path_meshes" value="package://panther_description/meshes"/>
-    <xacro:property name="M_PI" value="3.14159"/>
-    <!-- Sprocket and gear properties -->
-    <xacro:property name="sprocket_radius" value="0.0325"/>
-    <xacro:property name="sprocket_leght"  value="0.05"/>
-    <xacro:property name="sprocket_teeth"  value="24"/>
-    <xacro:property name="gear_teeth"      value="16"/>
-    <xacro:property name="wheel_offset_x"  value="-0.00"/>
-    <xacro:property name="wheel_offset_y"  value="0.08"/>
-    <xacro:property name="wheel_offset_z"  value="${wheel_radius}"/>
-    <xacro:property name="mboard" value="$(arg motor_board)"/>
-    <!-- base_link -->
-    <link name="base_link">
-        <visual>
-            <origin xyz="0 0 0" rpy="0 0 0" />
-            <geometry><cylinder length="0.001" radius="0.05"/></geometry>
-            <material name="Green" />
-        </visual>
-    </link>
-    <!-- Panther body -->
-    <xacro:chassis parent="base_link">
-        <origin xyz="0 0 0.08" rpy="0 0 0" />
-    </xacro:chassis>
-    <xacro:track type="left" parent="frame_link" />
-    <xacro:track type="right" parent="frame_link" />
-    <xacro:stand parent="frame_link" model="stand_rplidar_zed">
-        <origin xyz="-0.03600 0 0.1700" rpy="0 0 0" />
-    </xacro:stand>
-    <xacro:battery parent="frame_link" mass="0.24981">
-        <origin xyz="-0.13 0 0.01" rpy="0 0 0" />
-    </xacro:battery>
-    <xacro:if value="$(arg ssd)">
-        <xacro:include filename="$(find panther_description)/urdf/chassis/ssd.urdf.xacro" />
-        <xacro:ssd parent="frame_link">
-            <origin xyz="0.0465 0.03075 0.04674" rpy="${M_PI} 0 ${M_PI}" />
-        </xacro:ssd>
-    </xacro:if>
-    <!-- Sensors -->
-    <xacro:ultrasounds name="SFR10_left" parent="frame_link">
-        <origin xyz="0.15 0.095 -0.015" rpy="0 0 0" />
-    </xacro:ultrasounds>
-    <xacro:ultrasounds name="SFR10_right" parent="frame_link">
-        <origin xyz="0.15 -0.095 -0.015" rpy="0 0 0" />
-    </xacro:ultrasounds>
-    <xacro:ultrasounds name="SFR10_rear" parent="frame_link">
-        <origin xyz="-0.15 0 -0.015" rpy="${M_PI} ${M_PI} 0" />
-    </xacro:ultrasounds>
-    <xacro:razor_imu parent="frame_link">
-        <origin xyz="-0.0420817256507905 0 0.091441320597534" rpy="0 ${M_PI/2} 0" />
-    </xacro:razor_imu>
-    <xacro:zed parent="stand_link" camera_name="$(arg zed_model)" camera_model="$(arg zed_model)">
-        <origin xyz="0.028 0 0.021" rpy="0 0 0" />
-    </xacro:zed>
-    <xacro:rplidar parent="stand_link">
-        <origin xyz="-0.03 0 0.02" rpy="0 0 0" />
-    </xacro:rplidar>
-    <!-- Boards -->
-    <xacro:jetson parent="frame_link" model="$(arg jetson)">
-        <origin xyz="0.08 0 0.05" rpy="0 0 0" />
-    </xacro:jetson>
-    <xacro:if value="${mboard == 'unav'}">
-        <xacro:include filename="$(find panther_description)/urdf/boards/unav.urdf.xacro" />
-        <xacro:unav parent="frame_link">
-            <origin xyz="-0.10 0 0.12" rpy="0 0 0" />
-        </xacro:unav>
-    </xacro:if>
-    <xacro:if value="${mboard == 'roboteq'}">
-        <xacro:include filename="$(find panther_description)/urdf/boards/roboteq.urdf.xacro" />
-        <xacro:roboteq parent="frame_link">
-            <origin xyz="-0.11 0 0.12" rpy="0 0 0" />
-        </xacro:roboteq>
-    </xacro:if>
+    <xacro:arg name="zed_model"    default="zed2"/> <!-- Follow zed_repository -->
+    <xacro:arg name="jetson"       default="xavier"/> <!-- options: tx, xavier -->
+    <xacro:arg name="motor_board"  default="roboteq"/> <!-- options: unav, roboteq -->
+    <xacro:arg name="ssd"          default="false"/>
+    <xacro:arg name="ultrasounds"  default="false"/>
+    <xacro:panther
+               zed_model="$(arg zed_model)"
+               jetson="$(arg jetson)"
+               motor_board="$(arg motor_board)"
+               ssd="$(arg ssd)"
+               ultrasounds="$(arg ultrasounds)" />
 </robot>

Commit message: Fix color https://github.com/rpanther/panther_simulation/issues/3

File: panther_description/urdf/boards/jetson.urdf.xacro (robot description, xacro)
@@ -33,4 +33,7 @@
     <xacro:macro name="jetson" params="parent model *joint_pose">
         <xacro:if value="${model == 'xavier'}">
+            <gazebo reference="jetson_carrier_link">
+              <material>Gazebo/Black</material>
+            </gazebo>
             <link name="jetson_carrier_link">
                 <visual>

File: panther_description/urdf/boards/roboteq.urdf.xacro (robot description, xacro)
@@ -27,4 +27,7 @@
 <robot xmlns:xacro="http://ros.org/wiki/xacro" name="roboteq">
     <xacro:macro name="roboteq" params="parent *joint_pose">
+        <gazebo reference="roboteq_link">
+          <material>Gazebo/Black</material>
+        </gazebo>
         <link name="roboteq_link">
             <visual>

File: panther_description/urdf/track/track.urdf.xacro (robot description, xacro)
@@ -37,24 +37,24 @@
     <xacro:property name="orientation" value="1"/>
   </xacro:if>
-  <gazebo reference="track_${type}_Link">
-    <material>Gazebo/White</material>
-  </gazebo>
-  <gazebo reference="fender_${type}_Link">
+  <gazebo reference="track_${type}_link">
+    <material>Gazebo/GreyTransparent</material>
+  </gazebo>
+  <gazebo reference="fender_${type}_link">
     <material>Gazebo/Black</material>
   </gazebo>
-  <gazebo reference="chain_${type}_Link">
+  <gazebo reference="chain_${type}_link">
     <material>Gazebo/DarkGrey</material>
   </gazebo>
-  <gazebo reference="rubber_${type}_Link">
+  <gazebo reference="rubber_${type}_link">
     <material>Gazebo/Black</material>
   </gazebo>
-  <gazebo reference="iron_${type}_Link">
+  <gazebo reference="iron_${type}_link">
     <material>Gazebo/Grey</material>
   </gazebo>
-  <gazebo reference="damper_${type}_Link">
+  <gazebo reference="damper_${type}_link">
     <material>Gazebo/Black</material>
   </gazebo>
-  <gazebo reference="damper_label_${type}_Link">
-    <material>Gazebo/Red</material>
+  <gazebo reference="damper_label_${type}_link">
+    <material>Gazebo/Purple</material>
   </gazebo>
   <!-- TRACK FIXED LINKS -->
@@ -81,5 +81,5 @@
     <axis xyz="0 0 0" />
   </joint>
-  <link name="iron_${type}_Link">
+  <link name="iron_${type}_link">
     <inertial>
       <origin xyz="0.028 0.026 0.011" rpy="0 0 0" />
@@ -100,8 +100,8 @@
     <origin xyz="0 0 0" rpy="0 0 0" />
     <parent link="track_${type}_link" />
-    <child link="iron_${type}_Link" />
-    <axis xyz="0 0 0" />
-  </joint>
-  <link name="damper_${type}_Link">
+    <child link="iron_${type}_link" />
+    <axis xyz="0 0 0" />
+  </joint>
+  <link name="damper_${type}_link">
     <inertial>
       <origin xyz="0.011 0.014 0.028" rpy="0 0 0" />
@@ -122,8 +122,8 @@
     <origin xyz="0 0 0" rpy="0 0 0" />
     <parent link="track_${type}_link" />
-    <child link="damper_${type}_Link" />
-    <axis xyz="0 0 0" />
-  </joint>
-  <link name="damper_label_${type}_Link">
+    <child link="damper_${type}_link" />
+    <axis xyz="0 0 0" />
+  </joint>
+  <link name="damper_label_${type}_link">
     <inertial>
       <origin xyz="0.0111 0.0137 0.0341" rpy="0 0 0" />
@@ -143,9 +143,9 @@
   <joint name="damper_label_${type}_joint" type="fixed">
     <origin xyz="0 0 0" rpy="0 0 0" />
-    <parent link="damper_${type}_Link" />
-    <child link="damper_label_${type}_Link" />
-    <axis xyz="0 0 0" />
-  </joint>
-  <link name="fender_${type}_Link">
+    <parent link="damper_${type}_link" />
+    <child link="damper_label_${type}_link" />
+    <axis xyz="0 0 0" />
+  </joint>
+  <link name="fender_${type}_link">
     <inertial>
       <origin xyz="-0.0044 0.0167 0.0872" rpy="0 0 0" />
@@ -166,8 +166,8 @@
     <origin xyz="0 0 0" rpy="0 0 0" />
     <parent link="track_${type}_link" />
-    <child link="fender_${type}_Link" />
-    <axis xyz="0 0 0" />
-  </joint>
-  <link name="chain_${type}_Link">
+    <child link="fender_${type}_link" />
+    <axis xyz="0 0 0" />
+  </joint>
+  <link name="chain_${type}_link">
     <inertial>
       <origin xyz="0.101 0.0001 -0.0026" rpy="0 0 0" />
@@ -188,8 +188,8 @@
     <origin xyz="0 0 0" rpy="0 0 0" />
     <parent link="track_${type}_link" />
-    <child link="chain_${type}_Link" />
-    <axis xyz="0 0 0" />
-  </joint>
-  <link name="rubber_${type}_Link">
+    <child link="chain_${type}_link" />
+    <axis xyz="0 0 0" />
+  </joint>
+  <link name="rubber_${type}_link">
     <inertial>
       <origin xyz="-0.0137 0 -0.0014" rpy="0 0 0" />
@@ -210,5 +210,5 @@
     <origin xyz="0 0 0" rpy="0 0 0" />
     <parent link="track_${type}_link" />
-    <child link="rubber_${type}_Link" />
+    <child link="rubber_${type}_link" />
     <axis xyz="0 0 0" />
   </joint>

File: panther_description/urdf/track/wheel.urdf.xacro (robot description, xacro)
@@ -61,5 +61,5 @@
   </joint>
   <gazebo reference="wheel_${type}_${conf}_Link">
-    <material>Gazebo/WhiteGlow</material>
+    <material>Gazebo/GreyTransparent</material>
   </gazebo>
   </xacro:macro>
